File: MattzoController_Signal_I2C/EAGLE/Output_v2_0.brd (EAGLE design)
At the start: 90 x 90 mm, 87 parts, among them IC3 74HC540N, IC4 74HC540N, X4 057-016-0

Commit message: Update Output_v2_0.brd
Parts:
- moved C2 2.84 mm to (68.6, 8.89), turned to 270 degrees
- moved C1 1.27 mm to (44.5, 8.89), turned to 180 degrees
- turned C7 to 0 degrees
Routing:
- net VCC5.1: track 0.00 -> 472.4 mm
- net GND2: track 0.00 -> 201.0 mm
- net N$82: track 0.00 -> 104.8 mm
- net N$84: track 0.00 -> 82.5 mm
- net N$71: track 0.00 -> 58.5 mm
- net N$65: track 0.00 -> 48.1 mm
- net N$83: track 0.00 -> 46.3 mm
- net N$38: track 0.00 -> 36.2 mm
- net N$63: track 0.00 -> 35.4 mm
- net N$68: track 0.00 -> 34.9 mm
- net N$29: track 0.00 -> 32.6 mm
- net N$5: track 0.00 -> 31.1 mm
- net N$60: track 0.00 -> 27.5 mm
- net N$31: track 0.00 -> 27.5 mm
- net N$2: track 0.00 -> 25.0 mm
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Other:
- board text added: "1"
- board text added: "4"
- board text added: "5"
- board text added: "8"
- board text added: "A"
- board text added: "B"
