File: MattzoController_Switch_I2C/EAGLE/PWM_v2_0.brd (EAGLE design)
At the start: 90 x 90 mm, 12 parts, among them X1 MSTBA2, X4 057-016-0

Commit message: Update PWM_v2_0.brd
Parts:
- moved JP1 98.4 mm to (44.5, 72.4)
- moved F2 63.0 mm to (55.9, 40.6), turned to 90 degrees
- moved U$2 7.41 mm to (38.1, 47.0)
- moved F1 2.54 mm to (45.7, 16.5)
- moved JP13 1.80 mm to (14.0, 71.1)
- moved JP14 1.80 mm to (14.0, 12.7)
- moved J3 1.80 mm to (22.7, 41.9)
- moved X1 1.27 mm to (45.7, 3.81)
- moved J2 1.27 mm to (67.4, 41.9)
- moved JP7 1.27 mm to (76.2, 12.7)
- moved JP8 1.27 mm to (76.2, 71.1)
Connections:
- net N$14: now also JP8.5
- net N$15: now also JP14.5
Routing:
- net N$14: track 0.00 -> 101.3 mm
- net N$15: track 21.4 -> 96.1 mm
- net N$5: track 186.5 -> 225.9 mm, vias 2 -> 0
- net N$7: track 226.4 -> 258.6 mm, vias 2 -> 0
- net N$12: track 0.00 -> 30.6 mm
- net N$11: track 211.9 -> 237.5 mm, vias 2 -> 0
- net N$6: track 189.2 -> 206.4 mm, vias 2 -> 0
- net N$3: track 203.5 -> 218.3 mm, vias 2 -> 0
- net N$20: track 0.00 -> 9.20 mm
- net N$19: track 0.00 -> 9.20 mm
- net N$17: track 0.00 -> 8.15 mm
- net N$13: track 0.00 -> 8.15 mm
- net N$21: track 0.00 -> 6.66 mm
- net N$2: track 50.1 -> 56.4 mm
- net N$4: track 0.00 -> 5.61 mm
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