File: MattzoController_Switch_I2C/EAGLE/PWM_v2_0.sch (EAGLE design)
At the start: 12 parts, among them X1 MSTBA2, X4 057-016-0

Commit message: Update PWM_v2_0.sch
Connections:
- net N$14: now also JP8.5
- net N$15: now also JP14.5
Changed lines of the file:
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@@
 <wire x1="20.32" y1="45.72" x2="20.32" y2="48.26" width="0.1524" layer="91"/>
 <junction x="17.78" y="45.72"/>
+<pinref part="JP8" gate="A" pin="5"/>
+<wire x1="127" y1="27.94" x2="137.16" y2="27.94" width="0.1524" layer="91"/>
+<junction x="127" y="27.94"/>
 </segment>
 </net>
@@
 <wire x1="30.48" y1="45.72" x2="30.48" y2="48.26" width="0.1524" layer="91"/>
 <junction x="27.94" y="45.72"/>
+<pinref part="JP14" gate="A" pin="5"/>
+<wire x1="127" y1="76.2" x2="137.16" y2="76.2" width="0.1524" layer="91"/>
+<junction x="127" y="76.2"/>
 </segment>
 </net>
