File: MattzoController_Switch_I2C/EAGLE/PWM_v2_1.brd (EAGLE design)
At the start: 90 x 90 mm, 12 parts, among them X1 MSTBA2, X4 057-016-0

Commit message: Update PWM_v2_1.brd
Connections:
- net N$1: now also U$2.OUTB-
- net N$12: now also U$2.OUTB+
- net N$8: now also U$2.INB-
- net N$9: now also U$2.INB+
Routing:
- net N$1: track 0.00 -> 76.2 mm
- net N$2: track 0.00 -> 46.2 mm
- net N$9: track 0.00 -> 29.6 mm
- net N$8: track 0.00 -> 23.6 mm
- net N$12: track 0.00 -> 14.4 mm
- net N$10: track 0.00 -> 12.7 mm
Changed lines of the file:
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@@
 <contactref element="J2" pad="2"/>
 <contactref element="U$2" pad="OUTA-"/>
-<wire x1="67.437" y1="43.61" x2="60.55" y2="60.63" width="0" layer="19" extent="1-1"/>
-<wire x1="22.733" y1="40.21" x2="60.55" y2="60.63" width="0" layer="19" extent="1-1"/>
+<contactref element="U$2" pad="OUTB-"/>
+<wire x1="61.82" y1="65.71" x2="61.82" y2="61.9" width="1.27" layer="1"/>
+<wire x1="61.82" y1="61.9" x2="60.55" y2="60.63" width="1.27" layer="1"/>
+<wire x1="60.55" y1="50.497" x2="67.437" y2="43.61" width="1.27" layer="1"/>
+<wire x1="60.55" y1="60.63" x2="60.55" y2="50.497" width="1.27" layer="1"/>
+<wire x1="60.55" y1="60.63" x2="53.26" y2="53.34" width="1.27" layer="1"/>
+<wire x1="53.26" y1="53.34" x2="30.48" y2="53.34" width="1.27" layer="1"/>
+<wire x1="30.48" y1="53.34" x2="26.67" y2="49.53" width="1.27" layer="1"/>
+<wire x1="24.97" y1="40.21" x2="22.733" y2="40.21" width="1.27" layer="1"/>
+<wire x1="26.67" y1="49.53" x2="26.67" y2="41.91" width="1.27" layer="1"/>
+<wire x1="26.67" y1="41.91" x2="24.97" y2="40.21" width="1.27" layer="1"/>
 </signal>
 <signal name="N$2">
@@
 <contactref element="J2" pad="1"/>
 <contactref element="F2" pad="1"/>
-<wire x1="33.02" y1="42.0878" x2="67.437" y2="40.11" width="0" layer="19" extent="1-1"/>
-<wire x1="22.733" y1="43.71" x2="33.02" y2="42.0878" width="0" layer="19" extent="1-1"/>
+<wire x1="33.02" y1="42.0878" x2="59.5122" y2="42.0878" width="1.27" layer="1"/>
+<wire x1="61.49" y1="40.11" x2="67.437" y2="40.11" width="1.27" layer="1"/>
+<wire x1="59.5122" y1="42.0878" x2="61.49" y2="40.11" width="1.27" layer="1"/>
+<wire x1="22.733" y1="43.71" x2="31.3978" y2="43.71" width="1.27" layer="16"/>
+<wire x1="31.3978" y1="43.71" x2="33.02" y2="42.0878" width="1.27" layer="16"/>
 </signal>
 <signal name="N$11">
@@
 <contactref element="X1" pad="2"/>
 <contactref element="U$2" pad="INA-"/>
-<wire x1="48.26" y1="8.89" x2="60.55" y2="20.1" width="0" layer="19" extent="1-1"/>
+<contactref element="U$2" pad="INB-"/>
+<wire x1="48.26" y1="8.89" x2="49.53" y2="10.16" width="1.27" layer="1"/>
+<wire x1="49.53" y1="10.16" x2="59.69" y2="10.16" width="1.27" layer="1"/>
+<wire x1="59.69" y1="10.16" x2="62.23" y2="12.7" width="1.27" layer="1"/>
+<wire x1="62.23" y1="12.7" x2="62.23" y2="13.34" width="1.27" layer="1"/>
+<wire x1="62.23" y1="13.34" x2="61.82" y2="13.75" width="1.27" layer="1"/>
+<wire x1="61.82" y1="13.75" x2="61.82" y2="18.83" width="1.27" layer="1"/>
+<wire x1="61.82" y1="18.83" x2="60.55" y2="20.1" width="1.27" layer="1"/>
 </signal>
 <signal name="N$9">
 <contactref element="U$2" pad="INA+"/>
 <contactref element="F1" pad="1"/>
-<wire x1="33.02" y1="37.9222" x2="42.48" y2="20.1" width="0" layer="19" extent="1-1"/>
+<contactref element="U$2" pad="INB+"/>
+<wire x1="41.21" y1="13.75" x2="42.48" y2="15.02" width="1.27" layer="1"/>
+<wire x1="42.48" y1="15.02" x2="42.48" y2="20.1" width="1.27" layer="1"/>
+<wire x1="42.48" y1="20.1" x2="40.86" y2="20.1" width="1.27" layer="1"/>
+<wire x1="40.86" y1="20.1" x2="33.02" y2="27.94" width="1.27" layer="1"/>
+<wire x1="33.02" y1="27.94" x2="33.02" y2="37.9222" width="1.27" layer="1"/>
 </signal>
 <signal name="N$10">
 <contactref element="F1" pad="2"/>
 <contactref element="X1" pad="1"/>
-<wire x1="43.18" y1="8.89" x2="33.02" y2="12.8778" width="0" layer="19" extent="1-1"/>
+<wire x1="43.18" y1="8.89" x2="35.56" y2="8.89" width="1.27" layer="1"/>
+<wire x1="35.56" y1="8.89" x2="33.02" y2="11.43" width="1.27" layer="1"/>
+<wire x1="33.02" y1="11.43" x2="33.02" y2="12.8778" width="1.27" layer="1"/>
 </signal>
 <signal name="N$12">
 <contactref element="U$2" pad="OUTA+"/>
 <contactref element="F2" pad="2"/>
-<wire x1="42.48" y1="60.63" x2="33.02" y2="67.1322" width="0" layer="19" extent="1-1"/>
+<contactref element="U$2" pad="OUTB+"/>
+<wire x1="33.02" y1="67.1322" x2="39.7878" y2="67.1322" width="1.27" layer="1"/>
+<wire x1="39.7878" y1="67.1322" x2="41.21" y2="65.71" width="1.27" layer="1"/>
+<wire x1="41.21" y1="65.71" x2="42.48" y2="64.44" width="1.27" layer="1"/>
+<wire x1="42.48" y1="64.44" x2="42.48" y2="60.63" width="1.27" layer="1"/>
 </signal>
 <signal name="N$14">
@@
 <wire x1="58.42" y1="69.85" x2="64.77" y2="76.2" width="0.508" layer="16"/>
 <wire x1="64.77" y1="76.2" x2="68.58" y2="76.2" width="0.508" layer="16"/>
-<wire x1="68.58" y1="76.2" x2="72.3646" y2="72.4154" width="0.508" layer="16"/>
-<wire x1="72.3646" y1="72.4154" x2="72.39" y2="72.4154" width="0.508" layer="16"/>
+<wire x1="68.58" y1="76.2" x2="72.39" y2="72.39" width="0.508" layer="16"/>
 <contactref element="JP8" pad="5"/>
-<wire x1="72.3646" y1="72.4154" x2="72.39" y2="72.39" width="0.508" layer="16"/>
 <wire x1="72.39" y1="72.39" x2="72.39" y2="71.12" width="0.508" layer="16"/>
-<wire x1="72.39" y1="71.12" x2="72.39" y2="12.7" width="0.508" layer="16"/>
+<wire x1="72.39" y1="71.12" x2="72.39" y2="12.7" width="0.508" layer="1"/>
 </signal>
 <signal name="N$15">

Commit message: Update PWM_v2_1.brd
Routing:
- net N$1: track 76.2 -> 74.9 mm
Changed lines of the file:
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@@
 </element>
 <element name="J2" library="microbuilder" package="TERMBLOCK_1X2-3.5MM" value="" x="67.437" y="41.91" smashed="yes" rot="R270"/>
-<element name="JP7" library="adafruit" package="1X06-CLEANBIG" value="" x="76.2" y="12.7" smashed="yes" rot="R180">
+<element name="JP7" library="adafruit" library_urn="urn:adsk.eagle:library:420" package="1X06-CLEANBIG" package3d_urn="urn:adsk.eagle:package:6240713/1" value="" x="76.2" y="12.7" smashed="yes" rot="R180">
 <attribute name="VALUE" x="83.82" y="15.875" size="1.27" layer="27" rot="R180"/>
 </element>
-<element name="JP8" library="adafruit" package="1X06-CLEANBIG" value="" x="76.2" y="71.12" smashed="yes" rot="R180">
+<element name="JP8" library="adafruit" library_urn="urn:adsk.eagle:library:420" package="1X06-CLEANBIG" package3d_urn="urn:adsk.eagle:package:6240713/1" value="" x="76.2" y="71.12" smashed="yes" rot="R180">
 <attribute name="VALUE" x="83.82" y="74.295" size="1.27" layer="27" rot="R180"/>
 </element>
 <element name="J3" library="microbuilder" package="TERMBLOCK_1X2-3.5MM" value="" x="22.733" y="41.91" smashed="yes" rot="R90"/>
-<element name="JP13" library="adafruit" package="1X06-CLEANBIG" value="" x="13.97" y="71.12" smashed="yes">
+<element name="JP13" library="adafruit" library_urn="urn:adsk.eagle:library:420" package="1X06-CLEANBIG" package3d_urn="urn:adsk.eagle:package:6240713/1" value="" x="13.97" y="71.12" smashed="yes">
 <attribute name="VALUE" x="6.35" y="67.945" size="1.27" layer="27"/>
 </element>
-<element name="JP14" library="adafruit" package="1X06-CLEANBIG" value="" x="13.97" y="12.7" smashed="yes">
+<element name="JP14" library="adafruit" library_urn="urn:adsk.eagle:library:420" package="1X06-CLEANBIG" package3d_urn="urn:adsk.eagle:package:6240713/1" value="" x="13.97" y="12.7" smashed="yes">
 <attribute name="VALUE" x="6.35" y="9.525" size="1.27" layer="27"/>
 </element>
@@
 <contactref element="U$2" pad="OUTA-"/>
 <contactref element="U$2" pad="OUTB-"/>
-<wire x1="61.82" y1="65.71" x2="61.82" y2="61.9" width="1.27" layer="1"/>
+<wire x1="61.82" y1="64.44" x2="61.82" y2="61.9" width="1.27" layer="1"/>
 <wire x1="61.82" y1="61.9" x2="60.55" y2="60.63" width="1.27" layer="1"/>
 <wire x1="60.55" y1="50.497" x2="67.437" y2="43.61" width="1.27" layer="1"/>
@@
 <contactref element="U$2" pad="OUTB+"/>
 <wire x1="33.02" y1="67.1322" x2="39.7878" y2="67.1322" width="1.27" layer="1"/>
-<wire x1="39.7878" y1="67.1322" x2="41.21" y2="65.71" width="1.27" layer="1"/>
-<wire x1="41.21" y1="65.71" x2="42.48" y2="64.44" width="1.27" layer="1"/>
-<wire x1="42.48" y1="64.44" x2="42.48" y2="60.63" width="1.27" layer="1"/>
+<wire x1="39.7878" y1="67.1322" x2="41.21" y2="64.44" width="1.27" layer="1"/>
+<wire x1="41.21" y1="64.44" x2="41.21" y2="61.9" width="1.27" layer="1"/>
+<wire x1="41.21" y1="61.9" x2="42.48" y2="60.63" width="1.27" layer="1"/>
 </signal>
 <signal name="N$14">
