File: MattzoController_Switch_I2C/EAGLE/CPU_v3_1.brd (EAGLE design)
At the start: 90 x 90 mm, 13 parts, among them X4 057-016-0

Commit message: Update CPU_v3_1.brd
Routing:
- net N$15: track 113.9 -> 112.7 mm
- net GND: track 204.9 -> 203.7 mm
Changed lines of the file:
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@@
 <contactref element="U$2" pad="OUTB-"/>
 <wire x1="85.95" y1="55.55" x2="87.22" y2="56.82" width="1.016" layer="1"/>
-<wire x1="87.22" y1="56.82" x2="87.22" y2="60.63" width="1.016" layer="1"/>
+<wire x1="87.22" y1="56.82" x2="87.22" y2="59.36" width="1.016" layer="1"/>
 <wire x1="41.91" y1="5.08" x2="72.39" y2="5.08" width="1.016" layer="1"/>
 <via x="72.39" y="5.08" extent="1-16" drill="0.35" diameter="1.3"/>
@@
 <wire x1="67.31" y1="22.86" x2="67.31" y2="48.26" width="0.254" layer="16"/>
 <wire x1="58.42" y1="60.96" x2="62.23" y2="60.96" width="0.2" layer="16"/>
-<wire x1="62.23" y1="60.96" x2="64.77" y2="58.42" width="0.2" layer="16"/>
-<wire x1="64.77" y1="58.42" x2="68.58" y2="58.42" width="0.2" layer="16"/>
-<wire x1="68.58" y1="58.42" x2="69.85" y2="57.15" width="0.2" layer="16"/>
+<wire x1="62.23" y1="60.96" x2="66.04" y2="57.15" width="0.2" layer="16"/>
+<wire x1="66.04" y1="57.15" x2="69.85" y2="57.15" width="0.2" layer="16"/>
 <wire x1="69.85" y1="57.15" x2="69.85" y2="55.88" width="0.2" layer="16"/>
 </signal>
@@
 <wire x1="66.04" y1="52.07" x2="67.88" y2="53.91" width="1.016" layer="1"/>
 <wire x1="67.88" y1="53.91" x2="67.88" y2="55.55" width="1.016" layer="1"/>
-<wire x1="67.88" y1="55.55" x2="67.88" y2="59.36" width="1.016" layer="1"/>
-<wire x1="67.88" y1="59.36" x2="66.61" y2="60.63" width="1.016" layer="1"/>
+<wire x1="67.88" y1="55.55" x2="67.88" y2="58.09" width="1.016" layer="1"/>
+<wire x1="67.88" y1="58.09" x2="66.61" y2="59.36" width="1.016" layer="1"/>
 </signal>
 </signals>
