File: MattzoStationController_I2C/EAGLE/Crossing_v1_0.brd (EAGLE design)
At the start: 90 x 90 mm, 57 parts, among them X1 MSTBA2, X4 057-016-0

Commit message: Update Crossing_v1_0.brd
Parts:
- removed JP21, JP22, JP23, JP24: (no value), jumper:JP2
Connections:
- removed net N$20: JP21.1, JP29.4
- removed net N$37: JP22.1, JP29.10
- removed net N$38: JP21.3, JP29.1
- removed net N$39: JP22.3, JP29.7
- removed net N$40: JP23.3, JP30.1
- removed net N$41: JP23.2, JP30.2
- removed net N$42: JP24.1, JP30.10
- removed net N$43: JP23.1, JP30.4
- removed net N$44: JP22.2, JP29.8
- removed net N$45: JP21.2, JP29.2
- removed net N$46: JP24.3, JP30.7
- removed net N$47: JP24.2, JP30.8
- net N$1: now also U$2.OUT-; no longer U$2.OUT+
- net N$2: now also U$2.OUT+; no longer U$2.OUT-
Routing:
- net N$2: track 52.1 -> 32.8 mm
- net N$1: track 39.5 -> 58.3 mm
- net N$38: track 11.2 -> 0.00 mm
- net N$40: track 11.2 -> 0.00 mm
- net N$43: track 10.5 -> 0.00 mm
- net N$42: track 10.5 -> 0.00 mm
- net N$46: track 10.5 -> 0.00 mm
- net N$39: track 9.42 -> 0.00 mm
- net N$37: track 9.42 -> 0.00 mm
- net N$20: track 9.42 -> 0.00 mm
- net N$41: track 9.20 -> 0.00 mm
- net N$45: track 8.67 -> 0.00 mm
- net N$47: track 7.93 -> 0.00 mm
- net N$44: track 6.88 -> 0.00 mm
Changed lines of the file:
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@@
 <attribute name="VALUE" x="14.605" y="27.94" size="1.27" layer="27" rot="R90"/>
-</element>
-<element name="JP21" library="jumper" library_urn="urn:adsk.eagle:library:252" package="JP2" package3d_urn="urn:adsk.eagle:package:15452/1" value="" x="2.54" y="15.24" smashed="yes" rot="R270">
-<attribute name="POPULARITY" value="34" x="2.54" y="15.24" size="1.778" layer="27" rot="R270" display="off"/>
-<attribute name="VALUE" x="-1.778" y="18.796" size="1.27" layer="27" ratio="10" rot="R270"/>
-</element>
-<element name="JP22" library="jumper" library_urn="urn:adsk.eagle:library:252" package="JP2" package3d_urn="urn:adsk.eagle:package:15452/1" value="" x="2.54" y="22.86" smashed="yes" rot="R270">
-<attribute name="POPULARITY" value="34" x="2.54" y="22.86" size="1.778" layer="27" rot="R270" display="off"/>
-<attribute name="VALUE" x="-1.778" y="26.416" size="1.27" layer="27" ratio="10" rot="R270"/>
-</element>
-<element name="JP23" library="jumper" library_urn="urn:adsk.eagle:library:252" package="JP2" package3d_urn="urn:adsk.eagle:package:15452/1" value="" x="2.54" y="30.48" smashed="yes" rot="R270">
-<attribute name="POPULARITY" value="34" x="2.54" y="30.48" size="1.778" layer="27" rot="R270" display="off"/>
-<attribute name="VALUE" x="-1.778" y="34.036" size="1.27" layer="27" ratio="10" rot="R270"/>
-</element>
-<element name="JP24" library="jumper" library_urn="urn:adsk.eagle:library:252" package="JP2" package3d_urn="urn:adsk.eagle:package:15452/1" value="" x="2.54" y="38.1" smashed="yes" rot="R270">
-<attribute name="POPULARITY" value="34" x="2.54" y="38.1" size="1.778" layer="27" rot="R270" display="off"/>
-<attribute name="VALUE" x="-1.778" y="41.656" size="1.27" layer="27" ratio="10" rot="R270"/>
 </element>
 </elements>
 <signals>
 <signal name="N$1">
+<contactref element="J2" pad="2"/>
+<contactref element="U$2" pad="OUT-"/>
+<wire x1="26.543" y1="38.94" x2="51.64" y2="38.94" width="1.016" layer="1"/>
+<wire x1="51.64" y1="38.94" x2="54.61" y2="41.91" width="1.016" layer="1"/>
+<wire x1="54.61" y1="41.91" x2="54.61" y2="70.38" width="1.016" layer="1"/>
+<wire x1="54.61" y1="70.38" x2="54.2" y2="70.79" width="1.016" layer="1"/>
+</signal>
+<signal name="N$2">
+<contactref element="J2" pad="1"/>
 <contactref element="U$2" pad="OUT+"/>
-<contactref element="J2" pad="2"/>
-<wire x1="26.543" y1="38.94" x2="24.56" y2="38.94" width="1.016" layer="1"/>
-<wire x1="24.56" y1="38.94" x2="24.13" y2="39.37" width="1.016" layer="1"/>
-<wire x1="24.13" y1="39.37" x2="24.13" y2="45.72" width="1.016" layer="1"/>
-<wire x1="37.4" y1="58.99" x2="37.4" y2="70.79" width="1.016" layer="1"/>
-<wire x1="24.13" y1="45.72" x2="37.4" y2="58.99" width="1.016" layer="1"/>
-</signal>
-<signal name="N$2">
-<contactref element="U$2" pad="OUT-"/>
-<contactref element="J2" pad="1"/>
-<wire x1="26.543" y1="42.44" x2="47.52" y2="42.44" width="1.016" layer="1"/>
-<wire x1="54.2" y1="49.12" x2="54.2" y2="70.79" width="1.016" layer="1"/>
-<wire x1="47.52" y1="42.44" x2="54.2" y2="49.12" width="1.016" layer="1"/>
+<wire x1="26.543" y1="42.44" x2="37.4" y2="53.297" width="1.016" layer="1"/>
+<wire x1="37.4" y1="53.297" x2="37.4" y2="70.79" width="1.016" layer="1"/>
 </signal>
 <signal name="N$11">
@@
 <wire x1="11.43" y1="68.58" x2="11.43" y2="69.85" width="0.254" layer="1"/>
 </signal>
-<signal name="N$42">
-<contactref element="JP24" pad="1"/>
-<contactref element="JP30" pad="10"/>
-<wire x1="2.54" y1="40.64" x2="7.62" y2="40.64" width="0.254" layer="1"/>
-<wire x1="7.62" y1="40.64" x2="11.43" y2="36.83" width="0.254" layer="1"/>
-</signal>
-<signal name="N$43">
-<contactref element="JP30" pad="4"/>
-<contactref element="JP23" pad="1"/>
-<wire x1="2.54" y1="33.02" x2="5.08" y2="30.48" width="0.254" layer="1"/>
-<wire x1="5.08" y1="30.48" x2="10.16" y2="30.48" width="0.254" layer="1"/>
-<wire x1="10.16" y1="30.48" x2="11.43" y2="31.75" width="0.254" layer="1"/>
-</signal>
-<signal name="N$20">
-<contactref element="JP21" pad="1"/>
-<contactref element="JP29" pad="4"/>
-<wire x1="2.54" y1="17.78" x2="10.16" y2="17.78" width="0.254" layer="1"/>
-<wire x1="10.16" y1="17.78" x2="11.43" y2="19.05" width="0.254" layer="1"/>
-</signal>
-<signal name="N$37">
-<contactref element="JP22" pad="1"/>
-<contactref element="JP29" pad="10"/>
-<wire x1="2.54" y1="25.4" x2="10.16" y2="25.4" width="0.254" layer="1"/>
-<wire x1="10.16" y1="25.4" x2="11.43" y2="24.13" width="0.254" layer="1"/>
-</signal>
-<signal name="N$38">
-<contactref element="JP21" pad="3"/>
-<contactref element="JP29" pad="1"/>
-<wire x1="11.43" y1="16.51" x2="11.43" y2="15.24" width="0.254" layer="1"/>
-<wire x1="11.43" y1="15.24" x2="8.89" y2="12.7" width="0.254" layer="1"/>
-<wire x1="8.89" y1="12.7" x2="2.54" y2="12.7" width="0.254" layer="1"/>
-</signal>
-<signal name="N$39">
-<contactref element="JP22" pad="3"/>
-<contactref element="JP29" pad="7"/>
-<wire x1="2.54" y1="20.32" x2="10.16" y2="20.32" width="0.254" layer="1"/>
-<wire x1="10.16" y1="20.32" x2="11.43" y2="21.59" width="0.254" layer="1"/>
-</signal>
-<signal name="N$40">
-<contactref element="JP23" pad="3"/>
-<contactref element="JP30" pad="1"/>
-<wire x1="2.54" y1="27.94" x2="3.81" y2="27.94" width="0.254" layer="1"/>
-<wire x1="3.81" y1="27.94" x2="5.08" y2="26.67" width="0.254" layer="1"/>
-<wire x1="5.08" y1="26.67" x2="10.16" y2="26.67" width="0.254" layer="1"/>
-<wire x1="10.16" y1="26.67" x2="11.43" y2="27.94" width="0.254" layer="1"/>
-<wire x1="11.43" y1="27.94" x2="11.43" y2="29.21" width="0.254" layer="1"/>
-</signal>
-<signal name="N$41">
-<contactref element="JP23" pad="2"/>
-<contactref element="JP30" pad="2"/>
-<wire x1="2.54" y1="30.48" x2="3.81" y2="30.48" width="0.254" layer="1"/>
-<wire x1="2.54" y1="30.48" x2="5.08" y2="27.94" width="0.254" layer="1"/>
-<wire x1="7.62" y1="27.94" x2="8.89" y2="29.21" width="0.254" layer="1"/>
-<wire x1="5.08" y1="27.94" x2="7.62" y2="27.94" width="0.254" layer="1"/>
-</signal>
-<signal name="N$44">
-<contactref element="JP22" pad="2"/>
-<contactref element="JP29" pad="8"/>
-<wire x1="2.54" y1="22.86" x2="7.62" y2="22.86" width="0.254" layer="1"/>
-<wire x1="7.62" y1="22.86" x2="8.89" y2="21.59" width="0.254" layer="1"/>
-</signal>
-<signal name="N$45">
-<contactref element="JP21" pad="2"/>
-<contactref element="JP29" pad="2"/>
-<wire x1="2.54" y1="15.24" x2="3.81" y2="15.24" width="0.254" layer="1"/>
-<wire x1="3.81" y1="15.24" x2="5.08" y2="13.97" width="0.254" layer="1"/>
-<wire x1="5.08" y1="13.97" x2="7.62" y2="13.97" width="0.254" layer="1"/>
-<wire x1="7.62" y1="13.97" x2="8.89" y2="15.24" width="0.254" layer="1"/>
-<wire x1="8.89" y1="15.24" x2="8.89" y2="16.51" width="0.254" layer="1"/>
-</signal>
-<signal name="N$46">
-<contactref element="JP24" pad="3"/>
-<contactref element="JP30" pad="7"/>
-<wire x1="2.54" y1="35.56" x2="5.08" y2="33.02" width="0.254" layer="1"/>
-<wire x1="5.08" y1="33.02" x2="10.16" y2="33.02" width="0.254" layer="1"/>
-<wire x1="10.16" y1="33.02" x2="11.43" y2="34.29" width="0.254" layer="1"/>
-</signal>
-<signal name="N$47">
-<contactref element="JP24" pad="2"/>
-<contactref element="JP30" pad="8"/>
-<wire x1="2.54" y1="38.1" x2="5.08" y2="35.56" width="0.254" layer="1"/>
-<wire x1="5.08" y1="35.56" x2="7.62" y2="35.56" width="0.254" layer="1"/>
-<wire x1="7.62" y1="35.56" x2="8.89" y2="34.29" width="0.254" layer="1"/>
-</signal>
 </signals>
