File: MattzoStationController_I2C/EAGLE/Crossing_v1_0.sch (EAGLE design)
At the start: 57 parts, among them X1 MSTBA2, X4 057-016-0

Commit message: Update Crossing_v1_0.sch
Parts:
- removed JP21, JP22, JP23, JP24: (no value), jumper:JP2E
Connections:
- removed net N$20: JP21.1, JP29.4
- removed net N$37: JP22.1, JP29.10
- removed net N$38: JP21.3, JP29.1
- removed net N$39: JP22.3, JP29.7
- removed net N$40: JP23.3, JP30.1
- removed net N$41: JP23.2, JP30.2
- removed net N$42: JP24.1, JP30.10
- removed net N$43: JP23.1, JP30.4
- removed net N$44: JP22.2, JP29.8
- removed net N$45: JP21.2, JP29.2
- removed net N$46: JP24.3, JP30.7
- removed net N$47: JP24.2, JP30.8
- net N$1: now also U$2.OUT-; no longer U$2.OUT+
- net N$2: now also U$2.OUT+; no longer U$2.OUT-
Changed lines of the file:
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@@
 <part name="JP29" library="microbuilder" deviceset="HEADER-3X04" device=""/>
 <part name="JP30" library="microbuilder" deviceset="HEADER-3X04" device=""/>
-<part name="JP21" library="jumper" library_urn="urn:adsk.eagle:library:252" deviceset="JP2E" device="" package3d_urn="urn:adsk.eagle:package:15452/1"/>
-<part name="JP22" library="jumper" library_urn="urn:adsk.eagle:library:252" deviceset="JP2E" device="" package3d_urn="urn:adsk.eagle:package:15452/1"/>
-<part name="JP23" library="jumper" library_urn="urn:adsk.eagle:library:252" deviceset="JP2E" device="" package3d_urn="urn:adsk.eagle:package:15452/1"/>
-<part name="JP24" library="jumper" library_urn="urn:adsk.eagle:library:252" deviceset="JP2E" device="" package3d_urn="urn:adsk.eagle:package:15452/1"/>
 </parts>
 <sheets>
@@
 <attribute name="VALUE" x="322.58" y="-55.88" size="1.27" layer="95"/>
 </instance>
-<instance part="JP21" gate="1" x="307.34" y="20.32" smashed="yes" rot="R90">
-<attribute name="NAME" x="307.34" y="16.51" size="1.778" layer="95" rot="R180"/>
-<attribute name="VALUE" x="307.34" y="26.035" size="1.778" layer="96" rot="R180"/>
-</instance>
-<instance part="JP22" gate="1" x="307.34" y="0" smashed="yes" rot="R90">
-<attribute name="NAME" x="307.34" y="-3.81" size="1.778" layer="95" rot="R180"/>
-<attribute name="VALUE" x="307.34" y="5.715" size="1.778" layer="96" rot="R180"/>
-</instance>
-<instance part="JP23" gate="1" x="307.34" y="-22.86" smashed="yes" rot="R90">
-<attribute name="NAME" x="307.34" y="-26.67" size="1.778" layer="95" rot="R180"/>
-<attribute name="VALUE" x="307.34" y="-17.145" size="1.778" layer="96" rot="R180"/>
-</instance>
-<instance part="JP24" gate="1" x="307.34" y="-43.18" smashed="yes" rot="R90">
-<attribute name="NAME" x="307.34" y="-46.99" size="1.778" layer="95" rot="R180"/>
-<attribute name="VALUE" x="307.34" y="-37.465" size="1.778" layer="96" rot="R180"/>
-</instance>
 </instances>
 <busses>
@@
 <net name="N$1" class="0">
 <segment>
-<wire x1="170.18" y1="81.28" x2="175.26" y2="81.28" width="0.1524" layer="91"/>
-<wire x1="175.26" y1="81.28" x2="175.26" y2="63.5" width="0.1524" layer="91"/>
+<pinref part="J2" gate="G$1" pin="2"/>
+<pinref part="U$2" gate="G$1" pin="OUT-"/>
+<wire x1="185.166" y1="68.58" x2="185.166" y2="81.28" width="0.1524" layer="91"/>
+<wire x1="185.166" y1="81.28" x2="170.18" y2="81.28" width="0.1524" layer="91"/>
+</segment>
+</net>
+<net name="N$2" class="0">
+<segment>
+<wire x1="170.18" y1="83.82" x2="177.8" y2="83.82" width="0.1524" layer="91"/>
+<wire x1="177.8" y1="83.82" x2="177.8" y2="63.5" width="0.1524" layer="91"/>
+<pinref part="J2" gate="G$1" pin="1"/>
 <pinref part="U$2" gate="G$1" pin="OUT+"/>
-<wire x1="185.166" y1="63.5" x2="175.26" y2="63.5" width="0.1524" layer="91"/>
-<pinref part="J2" gate="G$1" pin="2"/>
-</segment>
-</net>
-<net name="N$2" class="0">
-<segment>
-<wire x1="170.18" y1="83.82" x2="177.8" y2="83.82" width="0.1524" layer="91"/>
-<wire x1="177.8" y1="83.82" x2="177.8" y2="68.58" width="0.1524" layer="91"/>
-<pinref part="U$2" gate="G$1" pin="OUT-"/>
-<wire x1="185.166" y1="68.58" x2="177.8" y2="68.58" width="0.1524" layer="91"/>
-<pinref part="J2" gate="G$1" pin="1"/>
+<wire x1="177.8" y1="63.5" x2="185.166" y2="63.5" width="0.1524" layer="91"/>
 </segment>
 </net>
@@
 </segment>
 </net>
-<net name="N$42" class="0">
-<segment>
-<pinref part="JP24" gate="1" pin="1"/>
-<pinref part="JP30" gate="G$1" pin="10"/>
-<wire x1="309.88" y1="-45.72" x2="327.66" y2="-45.72" width="0.1524" layer="91"/>
-</segment>
-</net>
-<net name="N$43" class="0">
-<segment>
-<pinref part="JP30" gate="G$1" pin="4"/>
-<pinref part="JP23" gate="1" pin="1"/>
-<wire x1="327.66" y1="-25.4" x2="309.88" y2="-25.4" width="0.1524" layer="91"/>
-</segment>
-</net>
-<net name="N$20" class="0">
-<segment>
-<pinref part="JP21" gate="1" pin="1"/>
-<pinref part="JP29" gate="G$1" pin="4"/>
-<wire x1="309.88" y1="17.78" x2="327.66" y2="17.78" width="0.1524" layer="91"/>
-</segment>
-</net>
-<net name="N$37" class="0">
-<segment>
-<pinref part="JP22" gate="1" pin="1"/>
-<pinref part="JP29" gate="G$1" pin="10"/>
-<wire x1="309.88" y1="-2.54" x2="327.66" y2="-2.54" width="0.1524" layer="91"/>
-</segment>
-</net>
-<net name="N$38" class="0">
-<segment>
-<pinref part="JP21" gate="1" pin="3"/>
-<pinref part="JP29" gate="G$1" pin="1"/>
-<wire x1="309.88" y1="22.86" x2="309.88" y2="27.94" width="0.1524" layer="91"/>
-<wire x1="309.88" y1="27.94" x2="327.66" y2="27.94" width="0.1524" layer="91"/>
-</segment>
-</net>
-<net name="N$39" class="0">
-<segment>
-<pinref part="JP22" gate="1" pin="3"/>
-<pinref part="JP29" gate="G$1" pin="7"/>
-<wire x1="309.88" y1="2.54" x2="309.88" y2="7.62" width="0.1524" layer="91"/>
-<wire x1="309.88" y1="7.62" x2="327.66" y2="7.62" width="0.1524" layer="91"/>
-</segment>
-</net>
-<net name="N$40" class="0">
-<segment>
-<pinref part="JP23" gate="1" pin="3"/>
-<pinref part="JP30" gate="G$1" pin="1"/>
-<wire x1="309.88" y1="-20.32" x2="309.88" y2="-15.24" width="0.1524" layer="91"/>
-<wire x1="309.88" y1="-15.24" x2="327.66" y2="-15.24" width="0.1524" layer="91"/>
-</segment>
-</net>
-<net name="N$41" class="0">
-<segment>
-<pinref part="JP23" gate="1" pin="2"/>
-<wire x1="309.88" y1="-22.86" x2="312.42" y2="-22.86" width="0.1524" layer="91"/>
-<wire x1="312.42" y1="-22.86" x2="312.42" y2="-17.78" width="0.1524" layer="91"/>
-<pinref part="JP30" gate="G$1" pin="2"/>
-<wire x1="312.42" y1="-17.78" x2="327.66" y2="-17.78" width="0.1524" layer="91"/>
-</segment>
-</net>
-<net name="N$44" class="0">
-<segment>
-<pinref part="JP22" gate="1" pin="2"/>
-<wire x1="309.88" y1="0" x2="312.42" y2="0" width="0.1524" layer="91"/>
-<wire x1="312.42" y1="0" x2="312.42" y2="5.08" width="0.1524" layer="91"/>
-<pinref part="JP29" gate="G$1" pin="8"/>
-<wire x1="312.42" y1="5.08" x2="327.66" y2="5.08" width="0.1524" layer="91"/>
-</segment>
-</net>
-<net name="N$45" class="0">
-<segment>
-<pinref part="JP21" gate="1" pin="2"/>
-<wire x1="309.88" y1="20.32" x2="312.42" y2="20.32" width="0.1524" layer="91"/>
-<wire x1="312.42" y1="20.32" x2="312.42" y2="25.4" width="0.1524" layer="91"/>
-<pinref part="JP29" gate="G$1" pin="2"/>
-<wire x1="312.42" y1="25.4" x2="327.66" y2="25.4" width="0.1524" layer="91"/>
-</segment>
-</net>
-<net name="N$46" class="0">
-<segment>
-<pinref part="JP24" gate="1" pin="3"/>
-<pinref part="JP30" gate="G$1" pin="7"/>
-<wire x1="309.88" y1="-40.64" x2="309.88" y2="-35.56" width="0.1524" layer="91"/>
-<wire x1="309.88" y1="-35.56" x2="327.66" y2="-35.56" width="0.1524" layer="91"/>
-</segment>
-</net>
-<net name="N$47" class="0">
-<segment>
-<pinref part="JP24" gate="1" pin="2"/>
-<wire x1="309.88" y1="-43.18" x2="312.42" y2="-43.18" width="0.1524" layer="91"/>
-<wire x1="312.42" y1="-43.18" x2="312.42" y2="-38.1" width="0.1524" layer="91"/>
-<pinref part="JP30" gate="G$1" pin="8"/>
-<wire x1="312.42" y1="-38.1" x2="327.66" y2="-38.1" width="0.1524" layer="91"/>
-</segment>
-</net>
