File: MCP23017 Boards/MCP23017_I16_v1_0.brd (EAGLE design)
At the start: 90 x 90 mm, 59 parts, among them IC3 74HC540N, IC4 74HC540N, IC5 MCP23017SP, X4 057-016-0

Commit message: Update MCP23017_I16_v1_0.brd
Parts:
- removed C3, C6: 100nF, resistor:C025-024X044
- removed IC1, IC2: (no value), uln-udn:DIL18
- removed IC3, IC4: 74HC540N, 74xx-eu:DIL20
Connections:
- removed net N$12: IC2.8, IC3.11
- removed net N$14: IC2.7, IC3.12
- removed net N$15: IC2.6, IC3.13
- removed net N$16: IC2.5, IC3.14
- removed net N$17: IC2.4, IC3.15
- removed net N$18: IC2.3, IC3.16
- removed net N$19: IC2.2, IC3.17
- removed net N$2 (its old number): IC2.17, IN_2.K, JP2.3
- removed net N$20: IC2.1, IC3.18
- removed net N$21: IC3.2, IC5.21
- removed net N$23: IC3.4, IC5.23
- removed net N$25: IC3.6, IC5.25
- removed net N$27: IC3.8, IC5.27
- removed net N$34: IC1.8, IC4.11
- removed net N$37: IC1.17, IN_10.K, JP18.3
- removed net N$39: IC1.7, IC4.12
- removed net N$4: IC2.15, IN_4.K, JP4.3
- removed net N$40: IC1.6, IC4.13
- removed net N$41: IC1.15, IN_12.K, JP20.3
- removed net N$43: IC1.13, IN_14.K, JP22.3
- removed net N$44: IC1.5, IC4.14
- removed net N$45: IC1.4, IC4.15
- removed net N$46: IC1.3, IC4.16
- removed net N$47: IC1.2, IC4.17
- removed net N$48: IC1.1, IC4.18
- removed net N$49: IC4.2, IC5.1
- removed net N$51: IC4.4, IC5.3
- removed net N$54: IC1.11, IN_16.K, JP24.3
- removed net N$55: IC4.6, IC5.5
- removed net N$57: IC4.8, IC5.7
- removed net N$7: IC2.13, IN_6.K, JP6.3
- removed net N$9: IC2.11, IN_8.K, JP8.3
- net GND1: no longer C3.1, C6.1, IC1.9, IC2.9, IC3.1, IC3.10, IC3.19, IC4.1, IC4.10, IC4.19
- net N$1: now also IC5.21; no longer IC2.18
- net N$22: now also IN_2.K, JP2.3; no longer IC3.3
- net N$24: now also IN_4.K, JP4.3; no longer IC3.5
- net N$26: now also IN_6.K, JP6.3; no longer IC3.7
- net N$28: now also IN_8.K, JP8.3; no longer IC3.9
- net N$3: now also IC5.23; no longer IC2.16
- net N$36: now also IC5.1; no longer IC1.18
- net N$38: now also IC5.3; no longer IC1.16
- net N$42: now also IC5.5; no longer IC1.14
- net N$5: now also IC5.25; no longer IC2.14
- net N$50: now also IN_10.K, JP18.3; no longer IC4.3
- net N$52: now also IN_12.K, JP20.3; no longer IC4.5
- net N$53: now also IC5.7; no longer IC1.12
- net N$56: now also IN_14.K, JP22.3; no longer IC4.7
- net N$58: now also IN_16.K, JP24.3; no longer IC4.9
- net N$8: now also IC5.27; no longer IC2.12
- net VCC5.2: no longer C3.2, C6.2, IC1.10, IC2.10, IC3.20, IC4.20
Routing:
- net VCC5.2: track 187.4 -> 0.00 mm
- net GND1: track 173.2 -> 0.00 mm
- net N$82: track 101.7 -> 0.00 mm
- net N$84: track 21.7 -> 0.00 mm
- net N$35: track 17.6 -> 0.00 mm
- net N$2: track 17.0 -> 0.00 mm
- net N$6: track 16.3 -> 1.27 mm
- net N$48: track 3.81 -> 0.00 mm
- net N$47: track 3.81 -> 0.00 mm
- net N$46: track 3.81 -> 0.00 mm
- net N$45: track 3.81 -> 0.00 mm
- net N$44: track 3.81 -> 0.00 mm
- net N$40: track 3.81 -> 0.00 mm
- net N$39: track 3.81 -> 0.00 mm
- net N$34: track 3.81 -> 0.00 mm
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Other:
- board text added: "MCP23017 I16 V1.0"
- board text removed: "1"
- board text removed: "4"
- board text removed: "5"
- board text removed: "8"
- board text removed: "A"
- board text removed: "B"
- board text removed: "Output V2.0"

Commit message: Update MCP23017_I16_v1_0.brd
Parts:
- moved C2 61.6 mm to (45.7, 66.0), turned to 0 degrees
- moved IC5 57.9 mm to (45.7, 44.5), turned to 270 degrees
- moved RN2 14.0 mm to (52.1, 21.6), turned to 0 degrees
- moved SW1 8.52 mm to (52.1, 11.4), turned to 0 degrees
Routing:
- net N$6: track 1.27 -> 5.68 mm

Commit message: Update MCP23017_I16_v1_0.brd
Parts:
- RN2: device resistor-net:RN-5 -> resistor-net_edit:RN-3
- moved IN_9 193.1 mm to (15.2, 78.7), turned to 180 degrees
- moved IN_8 188.8 mm to (73.7, 73.7)
- moved IN_7 182.0 mm to (73.7, 64.8)
- moved IN_6 175.9 mm to (73.7, 55.9)
- moved IN_5 170.5 mm to (73.7, 47.0)
- moved IN_10 170.2 mm to (15.2, 69.8), turned to 180 degrees
- moved IN_11 167.8 mm to (15.2, 61.0), turned to 180 degrees
- moved IN_4 165.9 mm to (73.7, 38.1)
- moved R18 153.7 mm to (11.4, 74.9)
- moved IN_12 152.7 mm to (15.2, 52.1), turned to 180 degrees
- moved R8 151.1 mm to (77.5, 68.6)
- moved JP8 145.1 mm to (86.4, 76.2), turned to 270 degrees
- moved IN_13 144.9 mm to (15.2, 43.2), turned to 180 degrees
- moved R20 141.1 mm to (11.4, 57.1)
- moved R7 139.8 mm to (77.5, 77.5)
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Routing:
- net VCC5.2: track 0.00 -> 380.1 mm
- net GND1: track 0.00 -> 363.0 mm
- net N$58: track 0.00 -> 66.1 mm
- net N$53: track 0.00 -> 60.0 mm
- net N$82: track 0.00 -> 57.7 mm, vias 0 -> 1
- net N$1: track 0.00 -> 56.7 mm
- net N$56: track 0.00 -> 56.6 mm
- net N$22: track 0.00 -> 52.6 mm
- net N$42: track 0.00 -> 52.5 mm
- net N$28: track 0.00 -> 50.3 mm
- net N$84: track 0.00 -> 50.1 mm
- net N$3: track 0.00 -> 48.4 mm
- net N$36: track 0.00 -> 48.4 mm
- net N$52: track 0.00 -> 48.4 mm
- net N$8: track 0.00 -> 47.0 mm
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Other:
- board text added: "By Djpredator69"
