File: MCP23017 Boards/MCP23017_O8_v1_0.sch (EAGLE design)
At the start: 83 parts, among them IC3 74HC540N, IC4 74HC540N, IC5 MCP23017SP, X4 057-016-0

Commit message: Update MCP23017_O8_v1_0.sch
Parts:
- removed C3, C6: 100nF, resistor:C-EU025-024X044
- removed IC1, IC2: (no value), uln-udn:ULN2803A
- removed IC3, IC4: 74HC540N, 74xx-eu:74HC540N
Connections:
- removed net N$12: IC2.I8, IC3A.Y8
- removed net N$14: IC2.I7, IC3A.Y7
- removed net N$15: IC2.I6, IC3A.Y6
- removed net N$16: IC2.I5, IC3A.Y5
- removed net N$17: IC2.I4, IC3A.Y4
- removed net N$18: IC2.I3, IC3A.Y3
- removed net N$19: IC2.I2, IC3A.Y2
- removed net N$2: IC2.O6, JP13.2, R1.2, R14.1
- removed net N$20: IC2.I1, IC3A.Y1
- removed net N$21: IC3A.A1, IC5.GPA0
- removed net N$23: IC3A.A3, IC5.GPA2
- removed net N$25: IC3A.A5, IC5.GPA4
- removed net N$27: IC3A.A7, IC5.GPA6
- removed net N$31: IC2.O2, JP16.2, R10.1, R3.2
- removed net N$34: IC1.I8, IC4A.Y8
- removed net N$38: IC2.O8, JP15.2, R16.1, R7.2
- removed net N$39: IC1.I7, IC4A.Y7
- removed net N$40: IC1.I6, IC4A.Y6
- removed net N$42: IC2.O4, JP11.2, R12.1, R5.2
- removed net N$44: IC1.I5, IC4A.Y5
- removed net N$45: IC1.I4, IC4A.Y4
- removed net N$46: IC1.I3, IC4A.Y3
- removed net N$47: IC1.I2, IC4A.Y2
- removed net N$48: IC1.I1, IC4A.Y1
- removed net N$50: IC4A.A2, IC5.GPB1
- removed net N$52: IC4A.A4, IC5.GPB3
- removed net N$55: IC4A.A5, IC5.GPB4
- removed net N$57: IC4A.A7, IC5.GPB6
- removed net N$59: IC1.O1, JP17.2, R18.2, R25.1
- removed net N$63: IC1.O3, JP18.2, R20.2, R27.1
- removed net N$68: IC1.O6, JP21.2, R21.2, R30.1
- removed net N$83: IC1.O8, JP23.2, R23.2, R32.1
- net GND2: no longer C3.1, C6.1, IC1.GND, IC2.GND, IC3A.G1, IC3A.G2, IC3P.GND, IC4A.G1, IC4A.G2, IC4P.GND
- net N$22: now also JP16.2, R10.1, R3.2; no longer IC3A.A2
- net N$24: now also JP11.2, R12.1, R5.2; no longer IC3A.A4
- net N$26: now also JP13.2, R1.2, R14.1; no longer IC3A.A6
- net N$28: now also JP15.2, R16.1, R7.2; no longer IC3A.A8
- net N$29: now also IC5.GPA0; no longer IC2.O1
- net N$41: now also IC5.GPA2; no longer IC2.O3
- net N$43: now also IC5.GPA4; no longer IC2.O5
- net N$49: now also JP17.2, R18.2, R25.1; no longer IC4A.A1
- net N$5: now also IC5.GPA6; no longer IC2.O7
- net N$51: now also JP18.2, R20.2, R27.1; no longer IC4A.A3
- net N$56: now also JP21.2, R21.2, R30.1; no longer IC4A.A6
- net N$58: now also JP23.2, R23.2, R32.1; no longer IC4A.A8
- net N$60: now also IC5.GPB1; no longer IC1.O2
- net N$64: now also IC5.GPB3; no longer IC1.O4
- net N$65: now also IC5.GPB4; no longer IC1.O5
- net N$71: now also IC5.GPB6; no longer IC1.O7
- net VCC5.1: no longer C3.2, C6.2, IC1.CD+, IC2.CD+, IC3P.VCC, IC4P.VCC
Other:
- moved on the sheet: JP1, JP10, JP11, JP12, JP13, JP14, JP15, JP16, JP17, JP18, JP19, JP2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

Commit message: Update MCP23017_O8_v1_0.sch
Parts:
- RN2: device resistor-net:RN04 -> resistor-net_edit:RN03
Changed lines of the file:
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@@
 <part name="JP24" library="jumper" library_urn="urn:adsk.eagle:library:252" deviceset="JP1E" device="" package3d_urn="urn:adsk.eagle:package:15455/1"/>
 <part name="SW1" library="special" library_urn="urn:adsk.eagle:library:367" deviceset="SW_DIP-3" device="" package3d_urn="urn:adsk.eagle:package:26663/2"/>
-<part name="RN2" library="resistor-net" library_urn="urn:adsk.eagle:library:343" deviceset="RN04" device="" package3d_urn="urn:adsk.eagle:package:24976/1"/>
+<part name="RN2" library="resistor-net_edit" deviceset="RN03" device=""/>
 <part name="IC5" library="microchip-6" deviceset="MCP23017" device="SP"/>
 </parts>
@@
 <attribute name="VALUE" x="78.74" y="-48.26" size="1.778" layer="96" rot="R180"/>
 </instance>
-<instance part="RN2" gate="1" x="81.28" y="-68.58" smashed="yes">
+<instance part="RN2" gate="G$1" x="81.28" y="-68.58" smashed="yes">
 <attribute name="NAME" x="78.74" y="-66.04" size="1.778" layer="95"/>
 <attribute name="VALUE" x="78.74" y="-72.898" size="1.778" layer="96"/>
@@
 <wire x1="33.02" y1="76.2" x2="60.96" y2="76.2" width="0.1524" layer="91"/>
 <junction x="33.02" y="83.82"/>
-<pinref part="RN2" gate="1" pin="1"/>
+<pinref part="RN2" gate="G$1" pin="1"/>
 <wire x1="76.2" y1="-68.58" x2="60.96" y2="-68.58" width="0.1524" layer="91"/>
 <pinref part="IC5" gate="G$1" pin="VSS"/>
@@
 <pinref part="SW1" gate="A" pin="4"/>
 <wire x1="81.28" y1="-58.42" x2="96.52" y2="-58.42" width="0.1524" layer="91"/>
-<pinref part="RN2" gate="1" pin="4"/>
+<pinref part="RN2" gate="G$1" pin="4"/>
 <wire x1="96.52" y1="-68.58" x2="96.52" y2="-58.42" width="0.1524" layer="91"/>
 <junction x="96.52" y="-58.42"/>
@@
 <pinref part="SW1" gate="A" pin="5"/>
 <wire x1="81.28" y1="-55.88" x2="91.44" y2="-55.88" width="0.1524" layer="91"/>
-<pinref part="RN2" gate="1" pin="3"/>
+<pinref part="RN2" gate="G$1" pin="3"/>
 <wire x1="91.44" y1="-68.58" x2="91.44" y2="-55.88" width="0.1524" layer="91"/>
 <junction x="91.44" y="-55.88"/>
@@
 <wire x1="86.36" y1="-53.34" x2="86.36" y2="-68.58" width="0.1524" layer="91"/>
 <junction x="86.36" y="-53.34"/>
-<pinref part="RN2" gate="1" pin="2"/>
-</segment>
-</net>
+<pinref part="RN2" gate="G$1" pin="2"/>
+</segment>
+</net>
