File: MCP23017 Boards/MCP23017_I8O4_v1_0.brd (EAGLE design)
At the start: 90 x 90 mm, 65 parts, among them IC5 MCP23017SP, X4 057-016-0

Commit message: Update MCP23017_I8O4_v1_0.brd
Routing:
- net VCC5.1: track 435.6 -> 415.8 mm
- net GND2: track 229.6 -> 218.7 mm
Changed lines of the file:
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@@
 </element>
 <element name="IC5" library="microchip-6" package="DIL28-3" value="MCP23017SP" x="45.72" y="44.45" smashed="yes" rot="R270">
-<attribute name="NAME" x="43.18" y="62.357" size="1.778" layer="25" ratio="10"/>
 <attribute name="VALUE" x="44.7802" y="60.198" size="1.778" layer="27" ratio="10" rot="R270"/>
 </element>
@@
 </element>
 <element name="JP1" library="jumper" library_urn="urn:adsk.eagle:library:252" package="JP2" package3d_urn="urn:adsk.eagle:package:15452/1" value="" x="85.09" y="13.97" smashed="yes" rot="R90">
-<attribute name="NAME" x="83.439" y="10.414" size="1.27" layer="25" ratio="10" rot="R90"/>
 <attribute name="POPULARITY" value="34" x="125.73" y="5.08" size="1.778" layer="27" rot="R90" display="off"/>
 <attribute name="VALUE" x="89.408" y="10.414" size="1.27" layer="27" ratio="10" rot="R90"/>
 </element>
 <element name="JP3" library="jumper" library_urn="urn:adsk.eagle:library:252" package="JP2" package3d_urn="urn:adsk.eagle:package:15452/1" value="" x="85.09" y="22.86" smashed="yes" rot="R90">
-<attribute name="NAME" x="83.439" y="19.304" size="1.27" layer="25" ratio="10" rot="R90"/>
 <attribute name="POPULARITY" value="34" x="125.73" y="-3.81" size="1.778" layer="27" rot="R90" display="off"/>
 <attribute name="VALUE" x="89.408" y="19.304" size="1.27" layer="27" ratio="10" rot="R90"/>
 </element>
 <element name="JP5" library="jumper" library_urn="urn:adsk.eagle:library:252" package="JP2" package3d_urn="urn:adsk.eagle:package:15452/1" value="" x="85.09" y="31.75" smashed="yes" rot="R90">
-<attribute name="NAME" x="83.439" y="28.194" size="1.27" layer="25" ratio="10" rot="R90"/>
 <attribute name="POPULARITY" value="34" x="125.73" y="-12.7" size="1.778" layer="27" rot="R90" display="off"/>
 <attribute name="VALUE" x="89.408" y="28.194" size="1.27" layer="27" ratio="10" rot="R90"/>
 </element>
 <element name="JP7" library="jumper" library_urn="urn:adsk.eagle:library:252" package="JP2" package3d_urn="urn:adsk.eagle:package:15452/1" value="" x="85.09" y="40.64" smashed="yes" rot="R90">
-<attribute name="NAME" x="83.439" y="37.084" size="1.27" layer="25" ratio="10" rot="R90"/>
 <attribute name="POPULARITY" value="34" x="125.73" y="-21.59" size="1.778" layer="27" rot="R90" display="off"/>
 <attribute name="VALUE" x="89.408" y="37.084" size="1.27" layer="27" ratio="10" rot="R90"/>
@@
 </element>
 <element name="JP10" library="jumper" library_urn="urn:adsk.eagle:library:252" package="JP2" package3d_urn="urn:adsk.eagle:package:15452/1" value="" x="85.09" y="58.42" smashed="yes" rot="R90">
-<attribute name="NAME" x="83.439" y="54.864" size="1.27" layer="25" ratio="10" rot="R90"/>
 <attribute name="POPULARITY" value="34" x="118.11" y="-3.81" size="1.778" layer="27" rot="R90" display="off"/>
 <attribute name="VALUE" x="89.408" y="54.864" size="1.27" layer="27" ratio="10" rot="R90"/>
 </element>
 <element name="JP11" library="jumper" library_urn="urn:adsk.eagle:library:252" package="JP2" package3d_urn="urn:adsk.eagle:package:15452/1" value="" x="85.09" y="67.31" smashed="yes" rot="R90">
-<attribute name="NAME" x="83.439" y="63.754" size="1.27" layer="25" ratio="10" rot="R90"/>
 <attribute name="POPULARITY" value="34" x="118.11" y="-12.7" size="1.778" layer="27" rot="R90" display="off"/>
 <attribute name="VALUE" x="89.408" y="63.754" size="1.27" layer="27" ratio="10" rot="R90"/>
 </element>
 <element name="JP12" library="jumper" library_urn="urn:adsk.eagle:library:252" package="JP2" package3d_urn="urn:adsk.eagle:package:15452/1" value="" x="85.09" y="76.2" smashed="yes" rot="R90">
-<attribute name="NAME" x="83.439" y="72.644" size="1.27" layer="25" ratio="10" rot="R90"/>
 <attribute name="POPULARITY" value="34" x="118.11" y="-21.59" size="1.778" layer="27" rot="R90" display="off"/>
 <attribute name="VALUE" x="89.408" y="72.644" size="1.27" layer="27" ratio="10" rot="R90"/>
@@
 <wire x1="85.09" y1="64.77" x2="88.476" y2="64.77" width="1.016" layer="1"/>
 <wire x1="85.09" y1="73.66" x2="88.476" y2="73.66" width="1.016" layer="1"/>
+<wire x1="41.91" y1="38.1" x2="43.18" y2="38.1" width="1.016" layer="16"/>
+<wire x1="46.99" y1="34.29" x2="46.99" y2="17.78" width="1.016" layer="16"/>
+<wire x1="43.18" y1="38.1" x2="46.99" y2="34.29" width="1.016" layer="16"/>
 <wire x1="85.09" y1="11.43" x2="59.69" y2="11.43" width="1.016" layer="16"/>
 <wire x1="59.69" y1="11.43" x2="57.15" y2="8.89" width="1.016" layer="16"/>
@@
 <wire x1="48.26" y1="8.89" x2="46.99" y2="10.16" width="1.016" layer="16"/>
 <wire x1="46.99" y1="10.16" x2="46.99" y2="17.78" width="1.016" layer="16"/>
-<wire x1="41.91" y1="38.1" x2="44.45" y2="38.1" width="0.508" layer="16"/>
-<wire x1="44.45" y1="38.1" x2="46.99" y2="40.64" width="0.508" layer="16"/>
-<wire x1="46.99" y1="40.64" x2="46.99" y2="68.58" width="0.508" layer="16"/>
 </signal>
 <signal name="VCC5.1">
@@
 <wire x1="1.524" y1="25.4" x2="1.524" y2="19.05" width="1.016" layer="16"/>
 <wire x1="1.524" y1="19.05" x2="1.524" y2="12.7" width="1.016" layer="16"/>
+<wire x1="1.524" y1="12.7" x2="1.524" y2="12.446" width="1.016" layer="16"/>
 <wire x1="3.81" y1="25.4" x2="1.524" y2="25.4" width="1.016" layer="16"/>
 <wire x1="3.81" y1="30.48" x2="1.524" y2="30.48" width="1.016" layer="16"/>
@@
 <wire x1="82.55" y1="5.08" x2="88.476" y2="11.006" width="1.016" layer="16"/>
 <wire x1="88.476" y1="11.006" x2="88.476" y2="13.546" width="1.016" layer="16"/>
-<wire x1="1.524" y1="12.7" x2="1.524" y2="11.176" width="1.016" layer="16"/>
+<wire x1="1.524" y1="12.446" x2="1.524" y2="11.176" width="1.016" layer="16"/>
 <wire x1="1.524" y1="11.176" x2="7.62" y2="5.08" width="1.016" layer="16"/>
 <wire x1="7.62" y1="5.08" x2="49.53" y2="5.08" width="1.016" layer="16"/>
@@
 <wire x1="52.07" y1="77.47" x2="49.53" y2="74.93" width="1.016" layer="16"/>
 <wire x1="49.53" y1="35.56" x2="48.26" y2="35.56" width="1.016" layer="16"/>
+<wire x1="48.26" y1="35.56" x2="46.99" y2="36.83" width="1.016" layer="16"/>
+<wire x1="46.99" y1="36.83" x2="46.99" y2="39.37" width="1.016" layer="16"/>
+<wire x1="46.99" y1="39.37" x2="45.72" y2="40.64" width="1.016" layer="16"/>
+<wire x1="45.72" y1="40.64" x2="41.91" y2="40.64" width="1.016" layer="16"/>
 <wire x1="85.09" y1="13.97" x2="64.77" y2="13.97" width="1.016" layer="16"/>
 <wire x1="60.96" y1="17.78" x2="60.96" y2="30.48" width="1.016" layer="16"/>
@@
 <wire x1="64.77" y1="13.97" x2="60.96" y2="17.78" width="1.016" layer="16"/>
 <wire x1="3.81" y1="12.7" x2="1.524" y2="12.7" width="1.016" layer="16"/>
-<wire x1="41.91" y1="40.64" x2="43.18" y2="40.64" width="0.508" layer="16"/>
-<wire x1="43.18" y1="40.64" x2="44.45" y2="41.91" width="0.508" layer="16"/>
-<wire x1="44.45" y1="41.91" x2="44.45" y2="68.58" width="0.508" layer="16"/>
 </signal>
 <signal name="N$59">
