File: MattzoController_Sensor_Digital_I2C/EAGLE/Input_v2_1.brd (EAGLE design)
At the start: 90 x 90 mm, 73 parts, among them X4 057-016-0

Commit message: Update Input_v2_1.brd
Parts:
- RN1, RN2: device resistor-net:RN-5 -> resistor-net_edit:RN-3
Changed lines of the file:
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@@
 <attribute name="VALUE" x="31.496" y="71.882" size="1.27" layer="27" ratio="10" rot="R270"/>
 </element>
-<element name="RN1" library="resistor-net" library_urn="urn:adsk.eagle:library:343" package="RN-5" package3d_urn="urn:adsk.eagle:package:24976/1" value="" x="45.72" y="67.31" smashed="yes" rot="R270">
+<element name="RN1" library="resistor-net_edit" package="RN-3" value="" x="45.72" y="67.31" smashed="yes" rot="R270">
 <attribute name="MF" value="" x="45.72" y="67.31" size="1.778" layer="27" rot="R270" display="off"/>
 <attribute name="MPN" value="" x="45.72" y="67.31" size="1.778" layer="27" rot="R270" display="off"/>
@@
 <attribute name="VALUE" x="42.799" y="71.12" size="1.27" layer="27" ratio="10" rot="R270"/>
 </element>
-<element name="RN2" library="resistor-net" library_urn="urn:adsk.eagle:library:343" package="RN-5" package3d_urn="urn:adsk.eagle:package:24976/1" value="" x="45.72" y="30.48" smashed="yes" rot="R270">
+<element name="RN2" library="resistor-net_edit" package="RN-3" value="" x="45.72" y="30.48" smashed="yes" rot="R270">
 <attribute name="MF" value="" x="45.72" y="30.48" size="1.778" layer="27" rot="R270" display="off"/>
 <attribute name="MPN" value="" x="45.72" y="30.48" size="1.778" layer="27" rot="R270" display="off"/>
