File: MattzoController_Sensor_Digital_I2C/EAGLE/Input_v2_1.sch (EAGLE design)
At the start: 73 parts, among them X4 057-016-0

Commit message: Update Input_v2_1.sch
Parts:
- RN1, RN2: device resistor-net:RN04 -> resistor-net_edit:RN03
Changed lines of the file:
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@@
 <part name="SW1" library="special" library_urn="urn:adsk.eagle:library:367" deviceset="SW_DIP-3" device="" package3d_urn="urn:adsk.eagle:package:26663/2"/>
 <part name="SW2" library="special" library_urn="urn:adsk.eagle:library:367" deviceset="SW_DIP-3" device="" package3d_urn="urn:adsk.eagle:package:26663/2"/>
-<part name="RN1" library="resistor-net" library_urn="urn:adsk.eagle:library:343" deviceset="RN04" device="" package3d_urn="urn:adsk.eagle:package:24976/1"/>
-<part name="RN2" library="resistor-net" library_urn="urn:adsk.eagle:library:343" deviceset="RN04" device="" package3d_urn="urn:adsk.eagle:package:24976/1"/>
+<part name="RN1" library="resistor-net_edit" deviceset="RN03" device=""/>
+<part name="RN2" library="resistor-net_edit" deviceset="RN03" device=""/>
 <part name="IN_1" library="led" library_urn="urn:adsk.eagle:library:259" deviceset="LED" device="3MM" package3d_urn="urn:adsk.eagle:package:15797/1"/>
 <part name="IN_2" library="led" library_urn="urn:adsk.eagle:library:259" deviceset="LED" device="3MM" package3d_urn="urn:adsk.eagle:package:15797/1"/>
@@
 <attribute name="VALUE" x="68.58" y="45.72" size="1.778" layer="96" rot="R180"/>
 </instance>
-<instance part="RN1" gate="1" x="68.58" y="66.04" smashed="yes">
+<instance part="RN1" gate="G$1" x="68.58" y="66.04" smashed="yes">
 <attribute name="NAME" x="66.04" y="68.58" size="1.778" layer="95"/>
 <attribute name="VALUE" x="66.04" y="61.722" size="1.778" layer="96"/>
 </instance>
-<instance part="RN2" gate="1" x="68.58" y="-35.56" smashed="yes">
+<instance part="RN2" gate="G$1" x="68.58" y="-35.56" smashed="yes">
 <attribute name="NAME" x="66.04" y="-33.02" size="1.778" layer="95"/>
 <attribute name="VALUE" x="66.04" y="-39.878" size="1.778" layer="96"/>
@@
 <wire x1="116.84" y1="73.66" x2="116.84" y2="58.42" width="0.1524" layer="91"/>
 <junction x="116.84" y="2.54"/>
-<pinref part="RN1" gate="1" pin="1"/>
+<pinref part="RN1" gate="G$1" pin="1"/>
 <wire x1="63.5" y1="66.04" x2="63.5" y2="73.66" width="0.1524" layer="91"/>
 <wire x1="63.5" y1="73.66" x2="116.84" y2="73.66" width="0.1524" layer="91"/>
-<pinref part="RN2" gate="1" pin="1"/>
+<pinref part="RN2" gate="G$1" pin="1"/>
 <wire x1="63.5" y1="-35.56" x2="63.5" y2="-27.94" width="0.1524" layer="91"/>
 <wire x1="63.5" y1="-27.94" x2="116.84" y2="-27.94" width="0.1524" layer="91"/>
@@
 <pinref part="U$1" gate="IC$1" pin="A2"/>
 <wire x1="71.12" y1="-66.04" x2="83.82" y2="-66.04" width="0.1524" layer="91"/>
-<pinref part="RN2" gate="1" pin="4"/>
+<pinref part="RN2" gate="G$1" pin="4"/>
 <wire x1="83.82" y1="-66.04" x2="91.44" y2="-66.04" width="0.1524" layer="91"/>
 <wire x1="83.82" y1="-35.56" x2="83.82" y2="-66.04" width="0.1524" layer="91"/>
@@
 <pinref part="U$1" gate="IC$1" pin="A1"/>
 <wire x1="71.12" y1="-63.5" x2="78.74" y2="-63.5" width="0.1524" layer="91"/>
-<pinref part="RN2" gate="1" pin="3"/>
+<pinref part="RN2" gate="G$1" pin="3"/>
 <wire x1="78.74" y1="-63.5" x2="91.44" y2="-63.5" width="0.1524" layer="91"/>
 <wire x1="78.74" y1="-35.56" x2="78.74" y2="-63.5" width="0.1524" layer="91"/>
@@
 <pinref part="SW1" gate="A" pin="6"/>
 <wire x1="91.44" y1="-60.96" x2="73.66" y2="-60.96" width="0.1524" layer="91"/>
-<pinref part="RN2" gate="1" pin="2"/>
+<pinref part="RN2" gate="G$1" pin="2"/>
 <wire x1="73.66" y1="-60.96" x2="71.12" y2="-60.96" width="0.1524" layer="91"/>
 <wire x1="73.66" y1="-35.56" x2="73.66" y2="-60.96" width="0.1524" layer="91"/>
@@
 <pinref part="U$4" gate="IC$1" pin="A0"/>
 <wire x1="71.12" y1="40.64" x2="73.66" y2="40.64" width="0.1524" layer="91"/>
-<pinref part="RN1" gate="1" pin="2"/>
+<pinref part="RN1" gate="G$1" pin="2"/>
 <wire x1="73.66" y1="40.64" x2="91.44" y2="40.64" width="0.1524" layer="91"/>
 <wire x1="73.66" y1="66.04" x2="73.66" y2="40.64" width="0.1524" layer="91"/>
@@
 <pinref part="U$4" gate="IC$1" pin="A1"/>
 <wire x1="71.12" y1="38.1" x2="78.74" y2="38.1" width="0.1524" layer="91"/>
-<pinref part="RN1" gate="1" pin="3"/>
+<pinref part="RN1" gate="G$1" pin="3"/>
 <wire x1="78.74" y1="38.1" x2="91.44" y2="38.1" width="0.1524" layer="91"/>
 <wire x1="78.74" y1="66.04" x2="78.74" y2="38.1" width="0.1524" layer="91"/>
@@
 <pinref part="U$4" gate="IC$1" pin="A2"/>
 <wire x1="71.12" y1="35.56" x2="83.82" y2="35.56" width="0.1524" layer="91"/>
-<pinref part="RN1" gate="1" pin="4"/>
+<pinref part="RN1" gate="G$1" pin="4"/>
 <wire x1="83.82" y1="35.56" x2="91.44" y2="35.56" width="0.1524" layer="91"/>
 <wire x1="83.82" y1="66.04" x2="83.82" y2="35.56" width="0.1524" layer="91"/>
