File: L9110 Board/EAGLE/L9110_v1_0.sch (EAGLE design)
At the start: 45 parts, among them IC5 MCP23017SP, X4 057-016-0

Commit message: Update L9110_v1_0.sch
Parts:
- added RN1: (no value), resistor-net_edit:RN08
Connections:
- net N$1: now also RN1.2
- net N$12: now also RN1.6
- net N$14: now also RN1.7
- net N$15: now also RN1.8
- net N$16: now also RN1.9
- net N$3: now also RN1.3
- net N$5: now also RN1.4
- net N$8: now also RN1.5
- net VCC5.1: now also RN1.1
