File: L9110 Board/EAGLE/L9110_v1_1.sch (EAGLE design)
At the start: 46 parts, among them IC5 MCP23017SP, X4 057-016-0

Commit message: Update L9110_v1_1.sch
Parts:
- U$2: value CP8-ADJ -> CP8-ADJ-B; device userlib:CP8-ADJ -> userlib:CP8-ADJ-B
Connections:
- net GND2: now also U$2.OUTA-; no longer U$2.OUT-
- net N$37: now also U$2.INA+; no longer U$2.IN+
- net N$38: now also U$2.INA-; no longer U$2.IN-
- net N$39: now also U$2.OUTA+; no longer U$2.OUT+
Changed lines of the file:
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@@
 <part name="C4" library="resistor" library_urn="urn:adsk.eagle:library:348" deviceset="C-EU" device="025-024X044" package3d_urn="urn:adsk.eagle:package:23630/1"/>
 <part name="C5" library="resistor" library_urn="urn:adsk.eagle:library:348" deviceset="C-EU" device="025-024X044" package3d_urn="urn:adsk.eagle:package:23630/1"/>
-<part name="U$2" library="userlib" deviceset="CP8-ADJ" device=""/>
+<part name="U$2" library="userlib" deviceset="CP8-ADJ-B" device=""/>
 <part name="6-12VDC" library="con-phoenix-508" library_urn="urn:adsk.eagle:library:176" deviceset="MSTBA2" device="" package3d_urn="urn:adsk.eagle:package:9615/1"/>
 <part name="F1" library="fuse" library_urn="urn:adsk.eagle:library:233" deviceset="SH22,5A" device="" package3d_urn="urn:adsk.eagle:package:14070/1"/>
@@
 <wire x1="251.46" y1="-91.44" x2="195.58" y2="-91.44" width="0.1524" layer="91"/>
 <junction x="195.58" y="-91.44"/>
-<pinref part="U$2" gate="G$1" pin="OUT-"/>
+<pinref part="U$2" gate="G$1" pin="OUTA-"/>
 <wire x1="231.394" y1="-106.68" x2="251.46" y2="-106.68" width="0.1524" layer="91"/>
 <wire x1="251.46" y1="-106.68" x2="251.46" y2="-91.44" width="0.1524" layer="91"/>
@@
 <net name="N$37" class="0">
 <segment>
-<pinref part="U$2" gate="G$1" pin="IN+"/>
+<pinref part="U$2" gate="G$1" pin="INA+"/>
 <pinref part="F1" gate="1" pin="1"/>
 <wire x1="200.914" y1="-101.6" x2="185.42" y2="-101.6" width="0.1524" layer="91"/>
@@
 <net name="N$38" class="0">
 <segment>
-<pinref part="U$2" gate="G$1" pin="IN-"/>
+<pinref part="U$2" gate="G$1" pin="INA-"/>
 <pinref part="6-12VDC" gate="-2" pin="1"/>
 <wire x1="200.914" y1="-106.68" x2="170.18" y2="-106.68" width="0.1524" layer="91"/>
@@
 <net name="N$39" class="0">
 <segment>
-<pinref part="U$2" gate="G$1" pin="OUT+"/>
+<pinref part="U$2" gate="G$1" pin="OUTA+"/>
 <pinref part="F2" gate="1" pin="2"/>
 <wire x1="231.394" y1="-101.6" x2="236.22" y2="-101.6" width="0.1524" layer="91"/>

Commit message: Update L9110_v1_1.sch
Connections:
- net GND2: now also U$2.OUTB-
- net N$37: now also U$2.INB+
- net N$38: now also U$2.INB-
- net N$39: now also U$2.OUTB+
Changed lines of the file:
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@@
 <wire x1="251.46" y1="-106.68" x2="251.46" y2="-91.44" width="0.1524" layer="91"/>
 <junction x="251.46" y="-91.44"/>
+<pinref part="U$2" gate="G$1" pin="OUTB-"/>
+<wire x1="231.14" y1="-109.22" x2="231.14" y2="-106.68" width="0.1524" layer="91"/>
+<wire x1="231.14" y1="-106.68" x2="231.394" y2="-106.68" width="0.1524" layer="91"/>
+<junction x="231.394" y="-106.68"/>
 </segment>
 </net>
@@
 <pinref part="F1" gate="1" pin="1"/>
 <wire x1="200.914" y1="-101.6" x2="185.42" y2="-101.6" width="0.1524" layer="91"/>
+<pinref part="U$2" gate="G$1" pin="INB+"/>
+<wire x1="200.66" y1="-99.06" x2="200.914" y2="-99.06" width="0.1524" layer="91"/>
+<wire x1="200.914" y1="-99.06" x2="200.914" y2="-101.6" width="0.1524" layer="91"/>
+<junction x="200.914" y="-101.6"/>
 </segment>
 </net>
@@
 <pinref part="6-12VDC" gate="-2" pin="1"/>
 <wire x1="200.914" y1="-106.68" x2="170.18" y2="-106.68" width="0.1524" layer="91"/>
+<pinref part="U$2" gate="G$1" pin="INB-"/>
+<wire x1="200.914" y1="-106.68" x2="200.914" y2="-109.22" width="0.1524" layer="91"/>
+<wire x1="200.914" y1="-109.22" x2="200.66" y2="-109.22" width="0.1524" layer="91"/>
+<junction x="200.914" y="-106.68"/>
 </segment>
 </net>
@@
 <pinref part="F2" gate="1" pin="2"/>
 <wire x1="231.394" y1="-101.6" x2="236.22" y2="-101.6" width="0.1524" layer="91"/>
-</segment>
-</net>
+<pinref part="U$2" gate="G$1" pin="OUTB+"/>
+<wire x1="231.394" y1="-101.6" x2="231.14" y2="-101.6" width="0.1524" layer="91"/>
+<wire x1="231.14" y1="-101.6" x2="231.14" y2="-99.06" width="0.1524" layer="91"/>
+<junction x="231.394" y="-101.6"/>
+</segment>
+</net>

Commit message: Update L9110_v1_1.sch
Parts:
- removed X1, X2, X3, X5: (no value), con-phoenix-254:MPT2
- added X6, X7, X8, X9: (no value), con-ptr500:AK300/2
Connections:
- net N$17: now also X6-2.KL; no longer X1-1.1
- net N$19: now also X6-1.KL; no longer X1-2.1
- net N$20: now also X7-2.KL; no longer X2-1.1
- net N$22: now also X7-1.KL; no longer X2-2.1
- net N$24: now also X8-2.KL; no longer X3-1.1
- net N$26: now also X8-1.KL; no longer X3-2.1
- net N$28: now also X9-2.KL; no longer X5-1.1
- net N$34: now also X9-1.KL; no longer X5-2.1
Changed lines of the file:
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@@
 <part name="F1" library="fuse" library_urn="urn:adsk.eagle:library:233" deviceset="SH22,5A" device="" package3d_urn="urn:adsk.eagle:package:14070/1"/>
 <part name="F2" library="fuse" library_urn="urn:adsk.eagle:library:233" deviceset="SH22,5A" device="" package3d_urn="urn:adsk.eagle:package:14070/1"/>
-<part name="X1" library="con-phoenix-254" library_urn="urn:adsk.eagle:library:172" deviceset="MPT2" device="" package3d_urn="urn:adsk.eagle:package:9320/1"/>
-<part name="X2" library="con-phoenix-254" library_urn="urn:adsk.eagle:library:172" deviceset="MPT2" device="" package3d_urn="urn:adsk.eagle:package:9320/1"/>
-<part name="X3" library="con-phoenix-254" library_urn="urn:adsk.eagle:library:172" deviceset="MPT2" device="" package3d_urn="urn:adsk.eagle:package:9320/1"/>
-<part name="X5" library="con-phoenix-254" library_urn="urn:adsk.eagle:library:172" deviceset="MPT2" device="" package3d_urn="urn:adsk.eagle:package:9320/1"/>
 <part name="RN1" library="resistor-net_edit" deviceset="RN08" device="" package3d_urn="urn:adsk.eagle:package:24977/1"/>
+<part name="X6" library="con-ptr500" library_urn="urn:adsk.eagle:library:181" deviceset="AK300/2" device="" package3d_urn="urn:adsk.eagle:package:9881/1"/>
+<part name="X7" library="con-ptr500" library_urn="urn:adsk.eagle:library:181" deviceset="AK300/2" device="" package3d_urn="urn:adsk.eagle:package:9881/1"/>
+<part name="X8" library="con-ptr500" library_urn="urn:adsk.eagle:library:181" deviceset="AK300/2" device="" package3d_urn="urn:adsk.eagle:package:9881/1"/>
+<part name="X9" library="con-ptr500" library_urn="urn:adsk.eagle:library:181" deviceset="AK300/2" device="" package3d_urn="urn:adsk.eagle:package:9881/1"/>
 </parts>
 <sheets>
@@
 <attribute name="VALUE" x="245.11" y="-98.679" size="1.778" layer="96" rot="R180"/>
 </instance>
-<instance part="X1" gate="-1" x="314.96" y="-12.7" smashed="yes">
-<attribute name="NAME" x="318.516" y="-13.335" size="1.778" layer="95"/>
-</instance>
-<instance part="X1" gate="-2" x="314.96" y="-20.32" smashed="yes">
-<attribute name="NAME" x="318.516" y="-20.955" size="1.778" layer="95"/>
-<attribute name="VALUE" x="313.944" y="-23.622" size="1.778" layer="96"/>
-</instance>
-<instance part="X2" gate="-1" x="314.96" y="-33.02" smashed="yes">
-<attribute name="NAME" x="318.516" y="-33.655" size="1.778" layer="95"/>
-</instance>
-<instance part="X2" gate="-2" x="314.96" y="-40.64" smashed="yes">
-<attribute name="NAME" x="318.516" y="-41.275" size="1.778" layer="95"/>
-<attribute name="VALUE" x="313.944" y="-43.942" size="1.778" layer="96"/>
-</instance>
-<instance part="X3" gate="-1" x="314.96" y="-53.34" smashed="yes">
-<attribute name="NAME" x="318.516" y="-53.975" size="1.778" layer="95"/>
-</instance>
-<instance part="X3" gate="-2" x="314.96" y="-60.96" smashed="yes">
-<attribute name="NAME" x="318.516" y="-61.595" size="1.778" layer="95"/>
-<attribute name="VALUE" x="313.944" y="-64.262" size="1.778" layer="96"/>
-</instance>
-<instance part="X5" gate="-1" x="314.96" y="-73.66" smashed="yes">
-<attribute name="NAME" x="318.516" y="-74.295" size="1.778" layer="95"/>
-</instance>
-<instance part="X5" gate="-2" x="314.96" y="-81.28" smashed="yes">
-<attribute name="NAME" x="318.516" y="-81.915" size="1.778" layer="95"/>
-<attribute name="VALUE" x="313.944" y="-84.582" size="1.778" layer="96"/>
-</instance>
 <instance part="RN1" gate="1" x="208.28" y="0" smashed="yes" rot="R270">
 <attribute name="NAME" x="210.82" y="2.54" size="1.778" layer="95" rot="R270"/>
 <attribute name="VALUE" x="203.962" y="2.54" size="1.778" layer="96" rot="R270"/>
+</instance>
+<instance part="X6" gate="-1" x="317.5" y="-20.32" smashed="yes" rot="R180">
+<attribute name="NAME" x="318.77" y="-21.209" size="1.778" layer="95"/>
+</instance>
+<instance part="X6" gate="-2" x="317.5" y="-12.7" smashed="yes" rot="R180">
+<attribute name="NAME" x="318.77" y="-13.589" size="1.778" layer="95"/>
+<attribute name="VALUE" x="321.31" y="-9.017" size="1.778" layer="96" rot="R180"/>
+</instance>
+<instance part="X7" gate="-1" x="317.5" y="-40.64" smashed="yes" rot="R180">
+<attribute name="NAME" x="318.77" y="-41.529" size="1.778" layer="95"/>
+</instance>
+<instance part="X7" gate="-2" x="317.5" y="-33.02" smashed="yes" rot="R180">
+<attribute name="NAME" x="318.77" y="-33.909" size="1.778" layer="95"/>
+<attribute name="VALUE" x="321.31" y="-29.337" size="1.778" layer="96" rot="R180"/>
+</instance>
+<instance part="X8" gate="-1" x="317.5" y="-60.96" smashed="yes" rot="R180">
+<attribute name="NAME" x="318.77" y="-61.849" size="1.778" layer="95"/>
+</instance>
+<instance part="X8" gate="-2" x="317.5" y="-53.34" smashed="yes" rot="R180">
+<attribute name="NAME" x="318.77" y="-54.229" size="1.778" layer="95"/>
+<attribute name="VALUE" x="321.31" y="-49.657" size="1.778" layer="96" rot="R180"/>
+</instance>
+<instance part="X9" gate="-1" x="317.5" y="-81.28" smashed="yes" rot="R180">
+<attribute name="NAME" x="318.77" y="-82.169" size="1.778" layer="95"/>
+</instance>
+<instance part="X9" gate="-2" x="317.5" y="-73.66" smashed="yes" rot="R180">
+<attribute name="NAME" x="318.77" y="-74.549" size="1.778" layer="95"/>
+<attribute name="VALUE" x="321.31" y="-69.977" size="1.778" layer="96" rot="R180"/>
 </instance>
 </instances>
@@
 <pinref part="C1" gate="G$1" pin="1"/>
 <wire x1="276.86" y1="-12.7" x2="299.72" y2="-12.7" width="0.1524" layer="91"/>
-<pinref part="X1" gate="-1" pin="1"/>
 <wire x1="299.72" y1="-12.7" x2="312.42" y2="-12.7" width="0.1524" layer="91"/>
 <junction x="299.72" y="-12.7"/>
+<pinref part="X6" gate="-2" pin="KL"/>
 </segment>
 </net>
@@
 <pinref part="IC1" gate="G$1" pin="1"/>
 <wire x1="299.72" y1="-20.32" x2="276.86" y2="-20.32" width="0.1524" layer="91"/>
-<pinref part="X1" gate="-2" pin="1"/>
 <wire x1="312.42" y1="-20.32" x2="299.72" y2="-20.32" width="0.1524" layer="91"/>
 <junction x="299.72" y="-20.32"/>
+<pinref part="X6" gate="-1" pin="KL"/>
 </segment>
 </net>
@@
 <pinref part="C3" gate="G$1" pin="1"/>
 <wire x1="276.86" y1="-33.02" x2="299.72" y2="-33.02" width="0.1524" layer="91"/>
-<pinref part="X2" gate="-1" pin="1"/>
 <wire x1="312.42" y1="-33.02" x2="299.72" y2="-33.02" width="0.1524" layer="91"/>
 <junction x="299.72" y="-33.02"/>
+<pinref part="X7" gate="-2" pin="KL"/>
 </segment>
 </net>
@@
 <pinref part="C3" gate="G$1" pin="2"/>
 <wire x1="276.86" y1="-40.64" x2="299.72" y2="-40.64" width="0.1524" layer="91"/>
-<pinref part="X2" gate="-2" pin="1"/>
 <wire x1="299.72" y1="-40.64" x2="312.42" y2="-40.64" width="0.1524" layer="91"/>
 <junction x="299.72" y="-40.64"/>
+<pinref part="X7" gate="-1" pin="KL"/>
 </segment>
 </net>
@@
 <pinref part="C4" gate="G$1" pin="1"/>
 <wire x1="276.86" y1="-53.34" x2="299.72" y2="-53.34" width="0.1524" layer="91"/>
-<pinref part="X3" gate="-1" pin="1"/>
 <wire x1="312.42" y1="-53.34" x2="299.72" y2="-53.34" width="0.1524" layer="91"/>
 <junction x="299.72" y="-53.34"/>
+<pinref part="X8" gate="-2" pin="KL"/>
 </segment>
 </net>
@@
 <pinref part="C4" gate="G$1" pin="2"/>
 <wire x1="276.86" y1="-60.96" x2="299.72" y2="-60.96" width="0.1524" layer="91"/>
-<pinref part="X3" gate="-2" pin="1"/>
 <wire x1="299.72" y1="-60.96" x2="312.42" y2="-60.96" width="0.1524" layer="91"/>
 <junction x="299.72" y="-60.96"/>
+<pinref part="X8" gate="-1" pin="KL"/>
 </segment>
 </net>
@@
 <pinref part="C5" gate="G$1" pin="1"/>
 <wire x1="276.86" y1="-73.66" x2="299.72" y2="-73.66" width="0.1524" layer="91"/>
-<pinref part="X5" gate="-1" pin="1"/>
 <wire x1="312.42" y1="-73.66" x2="299.72" y2="-73.66" width="0.1524" layer="91"/>
 <junction x="299.72" y="-73.66"/>
+<pinref part="X9" gate="-2" pin="KL"/>
 </segment>
 </net>
@@
 <pinref part="C5" gate="G$1" pin="2"/>
 <wire x1="276.86" y1="-81.28" x2="299.72" y2="-81.28" width="0.1524" layer="91"/>
-<pinref part="X5" gate="-2" pin="1"/>
 <wire x1="299.72" y1="-81.28" x2="312.42" y2="-81.28" width="0.1524" layer="91"/>
 <junction x="299.72" y="-81.28"/>
-</segment>
-</net>
+<pinref part="X9" gate="-1" pin="KL"/>
+</segment>
+</net>
