File: L9110 Board/EAGLE/L9110_v1_1.brd (EAGLE design)
At the start: 90 x 90 mm, 46 parts, among them IC5 MCP23017SP, X4 057-016-0

Commit message: Update L9110_v1_1.brd
Parts:
- U$2: value CP8-ADJ -> CP8-ADJ-B; device userlib:CP8-ADJ -> userlib:CP8-ADJ-B
- moved RN1 15.7 mm to (41.9, 66.0)
- moved IC5 15.3 mm to (53.3, 57.1)
- moved SW1 11.7 mm to (72.4, 8.89), turned to 90 degrees
- moved C2 8.98 mm to (53.3, 76.2)
- moved RN2 6.84 mm to (63.5, 8.89), turned to 90 degrees
- moved F2 4.58 mm to (33.0, 57.1)
- moved C3 3.81 mm to (12.7, 67.3)
- moved C4 3.81 mm to (12.7, 55.9)
- moved C5 3.81 mm to (12.7, 44.5)
- moved IC2 3.81 mm to (20.3, 67.3)
- moved IC3 3.81 mm to (20.3, 55.9)
- moved IC4 3.81 mm to (20.3, 44.5)
- moved X2 3.81 mm to (3.81, 67.3)
- moved X3 3.81 mm to (3.81, 55.9)
- moved X5 3.81 mm to (3.81, 44.5)
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Connections:
- net GND2: now also U$2.OUTA-; no longer U$2.OUT-
- net N$37: now also U$2.INA+; no longer U$2.IN+
- net N$38: now also U$2.INA-; no longer U$2.IN-
- net N$39: now also U$2.OUTA+; no longer U$2.OUT+
Routing:
- net GND2: track 306.3 -> 0.00 mm
- net VCC5.1: track 249.4 -> 0.00 mm
- net N$18: track 93.1 -> 0.00 mm
- net N$82: track 65.3 -> 0.00 mm
- net N$84: track 62.7 -> 0.00 mm
- net VCC5.2: track 62.2 -> 0.00 mm
- net N$38: track 46.2 -> 0.00 mm
- net N$21: track 43.4 -> 0.00 mm
- net N$9: track 42.5 -> 0.00 mm
- net N$3: track 38.8 -> 0.00 mm
- net N$2: track 37.8 -> 0.00 mm
- net N$1: track 37.4 -> 0.00 mm
- net N$27: track 36.2 -> 0.00 mm
- net N$23: track 33.6 -> 0.00 mm
- net N$8: track 32.5 -> 0.00 mm
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Other:
- board text added: "L9110 V1.1"
- board text removed: "L9110 V1.0"

Commit message: Update L9110_v1_1.brd
Connections:
- net GND2: now also U$2.OUTB-
- net N$37: now also U$2.INB+
- net N$38: now also U$2.INB-
- net N$39: now also U$2.OUTB+
Routing:
- net GND2: track 0.00 -> 322.9 mm, vias 0 -> 1
- net VCC5.1: track 0.00 -> 186.8 mm
- net N$18: track 0.00 -> 85.9 mm
- net N$21: track 0.00 -> 64.2 mm
- net VCC5.2: track 0.00 -> 62.2 mm
- net N$2: track 0.00 -> 61.9 mm
- net N$23: track 0.00 -> 57.8 mm
- net N$4: track 0.00 -> 49.9 mm
- net N$38: track 0.00 -> 49.8 mm
- net N$82: track 0.00 -> 49.3 mm
- net N$84: track 0.00 -> 45.3 mm
- net N$6: track 0.00 -> 45.0 mm
- net N$35: track 0.00 -> 44.2 mm
- net N$85: track 0.00 -> 43.5 mm
- net N$25: track 0.00 -> 38.8 mm
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
Commit message: Update L9110_v1_1.brd
Parts:
- removed X1, X2, X3, X5: (no value), con-phoenix-254:2POL254
- added X6, X7, X8, X9: (no value), con-ptr500:AK300/2
Connections:
- net N$17: now also X6.2; no longer X1.1
- net N$19: now also X6.1; no longer X1.2
- net N$20: now also X7.2; no longer X2.1
- net N$22: now also X7.1; no longer X2.2
- net N$24: now also X8.2; no longer X3.1
- net N$26: now also X8.1; no longer X3.2
- net N$28: now also X9.2; no longer X5.1
- net N$34: now also X9.1; no longer X5.2
Routing:
- net N$34: track 13.8 -> 4.86 mm
- net N$28: track 13.8 -> 4.86 mm
- net N$26: track 13.8 -> 4.86 mm
- net N$24: track 13.8 -> 4.86 mm
- net N$22: track 13.8 -> 4.86 mm
- net N$20: track 13.8 -> 4.86 mm
- net N$19: track 13.8 -> 4.86 mm
- net N$17: track 13.8 -> 4.86 mm

Commit message: Update L9110_v1_1.brd
Routing:
- net N$22: track 4.86 -> 13.0 mm
- net N$34: track 4.86 -> 13.0 mm
- net N$26: track 4.86 -> 13.0 mm
- net N$19: track 4.86 -> 13.0 mm
- net N$28: track 4.86 -> 13.0 mm
- net N$24: track 4.86 -> 13.0 mm
- net N$20: track 4.86 -> 13.0 mm
- net N$17: track 4.86 -> 13.0 mm
- net N$39: track 26.5 -> 25.2 mm
- net GND2: track 322.9 -> 322.2 mm
Changed lines of the file:
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@@
 <element name="IN_1" library="led" library_urn="urn:adsk.eagle:library:259" package="LED3MM" package3d_urn="urn:adsk.eagle:package:15797/1" value="" x="80.01" y="17.78" smashed="yes" rot="R270">
 <attribute name="NAME" x="80.391" y="15.875" size="1.27" layer="25" ratio="10" rot="R270"/>
+<attribute name="POPULARITY" value="97" x="80.01" y="17.78" size="1.778" layer="27" rot="R270" display="off"/>
 <attribute name="VALUE" x="78.359" y="15.875" size="1.27" layer="27" ratio="10" rot="R270"/>
 </element>
 <element name="IN_2" library="led" library_urn="urn:adsk.eagle:library:259" package="LED3MM" package3d_urn="urn:adsk.eagle:package:15797/1" value="" x="80.01" y="26.67" smashed="yes" rot="R270">
 <attribute name="NAME" x="80.391" y="24.765" size="1.27" layer="25" ratio="10" rot="R270"/>
+<attribute name="POPULARITY" value="97" x="80.01" y="26.67" size="1.778" layer="27" rot="R270" display="off"/>
 <attribute name="VALUE" x="78.359" y="24.765" size="1.27" layer="27" ratio="10" rot="R270"/>
 </element>
 <element name="IN_3" library="led" library_urn="urn:adsk.eagle:library:259" package="LED3MM" package3d_urn="urn:adsk.eagle:package:15797/1" value="" x="80.01" y="35.56" smashed="yes" rot="R270">
 <attribute name="NAME" x="80.391" y="33.655" size="1.27" layer="25" ratio="10" rot="R270"/>
+<attribute name="POPULARITY" value="97" x="80.01" y="35.56" size="1.778" layer="27" rot="R270" display="off"/>
 <attribute name="VALUE" x="78.359" y="33.655" size="1.27" layer="27" ratio="10" rot="R270"/>
 </element>
 <element name="IN_4" library="led" library_urn="urn:adsk.eagle:library:259" package="LED3MM" package3d_urn="urn:adsk.eagle:package:15797/1" value="" x="80.01" y="44.45" smashed="yes" rot="R270">
 <attribute name="NAME" x="80.391" y="42.545" size="1.27" layer="25" ratio="10" rot="R270"/>
+<attribute name="POPULARITY" value="97" x="80.01" y="44.45" size="1.778" layer="27" rot="R270" display="off"/>
 <attribute name="VALUE" x="78.359" y="42.545" size="1.27" layer="27" ratio="10" rot="R270"/>
 </element>
 <element name="IN_5" library="led" library_urn="urn:adsk.eagle:library:259" package="LED3MM" package3d_urn="urn:adsk.eagle:package:15797/1" value="" x="80.01" y="53.34" smashed="yes" rot="R270">
 <attribute name="NAME" x="80.391" y="51.435" size="1.27" layer="25" ratio="10" rot="R270"/>
+<attribute name="POPULARITY" value="97" x="80.01" y="53.34" size="1.778" layer="27" rot="R270" display="off"/>
 <attribute name="VALUE" x="78.359" y="51.435" size="1.27" layer="27" ratio="10" rot="R270"/>
 </element>
 <element name="IN_6" library="led" library_urn="urn:adsk.eagle:library:259" package="LED3MM" package3d_urn="urn:adsk.eagle:package:15797/1" value="" x="80.01" y="62.23" smashed="yes" rot="R270">
 <attribute name="NAME" x="80.391" y="60.325" size="1.27" layer="25" ratio="10" rot="R270"/>
+<attribute name="POPULARITY" value="97" x="80.01" y="62.23" size="1.778" layer="27" rot="R270" display="off"/>
 <attribute name="VALUE" x="78.359" y="60.325" size="1.27" layer="27" ratio="10" rot="R270"/>
 </element>
 <element name="IN_7" library="led" library_urn="urn:adsk.eagle:library:259" package="LED3MM" package3d_urn="urn:adsk.eagle:package:15797/1" value="" x="80.01" y="71.12" smashed="yes" rot="R270">
 <attribute name="NAME" x="80.391" y="69.215" size="1.27" layer="25" ratio="10" rot="R270"/>
+<attribute name="POPULARITY" value="97" x="80.01" y="71.12" size="1.778" layer="27" rot="R270" display="off"/>
 <attribute name="VALUE" x="78.359" y="69.215" size="1.27" layer="27" ratio="10" rot="R270"/>
 </element>
 <element name="IN_8" library="led" library_urn="urn:adsk.eagle:library:259" package="LED3MM" package3d_urn="urn:adsk.eagle:package:15797/1" value="" x="80.01" y="80.01" smashed="yes" rot="R270">
 <attribute name="NAME" x="80.391" y="78.105" size="1.27" layer="25" ratio="10" rot="R270"/>
+<attribute name="POPULARITY" value="97" x="80.01" y="80.01" size="1.778" layer="27" rot="R270" display="off"/>
 <attribute name="VALUE" x="78.359" y="78.105" size="1.27" layer="27" ratio="10" rot="R270"/>
 </element>
@@
 <contactref element="U$2" pad="OUTA-"/>
 <contactref element="U$2" pad="OUTB-"/>
-<wire x1="49.53" y1="17.33" x2="53.34" y2="17.33" width="1.016" layer="1"/>
-<wire x1="53.34" y1="17.33" x2="54.61" y2="16.06" width="1.016" layer="1"/>
+<wire x1="49.53" y1="17.33" x2="52.07" y2="17.33" width="1.016" layer="1"/>
+<wire x1="52.07" y1="17.33" x2="53.34" y2="16.06" width="1.016" layer="1"/>
 <wire x1="24.13" y1="82.55" x2="21.59" y2="82.55" width="1.016" layer="16"/>
 <wire x1="21.59" y1="82.55" x2="21.59" y2="74.93" width="1.016" layer="16"/>
@@
 <wire x1="28.39" y1="17.33" x2="49.53" y2="17.33" width="1.016" layer="16"/>
 <wire x1="21.59" y1="24.13" x2="28.39" y2="17.33" width="1.016" layer="16"/>
-<wire x1="54.61" y1="16.06" x2="54.61" y2="7.62" width="0.508" layer="16"/>
-<wire x1="54.61" y1="7.62" x2="58.42" y2="3.81" width="0.508" layer="16"/>
+<wire x1="53.34" y1="16.06" x2="53.34" y2="8.89" width="0.508" layer="16"/>
+<wire x1="53.34" y1="8.89" x2="58.42" y2="3.81" width="0.508" layer="16"/>
 <wire x1="58.42" y1="3.81" x2="63.5" y2="3.81" width="0.508" layer="16"/>
 <wire x1="85.09" y1="11.43" x2="85.09" y2="7.62" width="0.508" layer="16"/>
@@
 <wire x1="15.24" y1="74.93" x2="12.7" y2="77.47" width="1.016" layer="1"/>
 <contactref element="X6" pad="2"/>
-<wire x1="5.08" y1="76.2508" x2="16.51" y2="74.93" width="0" layer="19" extent="1-1"/>
+<wire x1="5.08" y1="76.2508" x2="11.4808" y2="76.2508" width="1.016" layer="1"/>
+<wire x1="11.4808" y1="76.2508" x2="12.7" y2="77.47" width="1.016" layer="1"/>
 </signal>
 <signal name="N$19">
@@
 <wire x1="15.24" y1="82.55" x2="12.7" y2="80.01" width="1.016" layer="1"/>
 <contactref element="X6" pad="1"/>
-<wire x1="5.08" y1="81.2546" x2="12.7" y2="80.01" width="0" layer="19" extent="1-1"/>
+<wire x1="5.08" y1="81.2546" x2="11.4554" y2="81.2546" width="1.016" layer="1"/>
+<wire x1="11.4554" y1="81.2546" x2="12.7" y2="80.01" width="1.016" layer="1"/>
 </signal>
 <signal name="N$20">
@@
 <wire x1="15.24" y1="63.5" x2="12.7" y2="66.04" width="1.016" layer="1"/>
 <contactref element="X7" pad="2"/>
-<wire x1="5.08" y1="64.8208" x2="16.51" y2="63.5" width="0" layer="19" extent="1-1"/>
+<wire x1="5.08" y1="64.8208" x2="11.4808" y2="64.8208" width="1.016" layer="1"/>
+<wire x1="11.4808" y1="64.8208" x2="12.7" y2="66.04" width="1.016" layer="1"/>
 </signal>
 <signal name="N$22">
@@
 <wire x1="15.24" y1="71.12" x2="12.7" y2="68.58" width="1.016" layer="1"/>
 <contactref element="X7" pad="1"/>
-<wire x1="5.08" y1="69.8246" x2="12.7" y2="68.58" width="0" layer="19" extent="1-1"/>
+<wire x1="5.08" y1="69.8246" x2="11.4554" y2="69.8246" width="1.016" layer="1"/>
+<wire x1="11.4554" y1="69.8246" x2="12.7" y2="68.58" width="1.016" layer="1"/>
 </signal>
 <signal name="N$24">
@@
 <wire x1="15.24" y1="52.07" x2="12.7" y2="54.61" width="1.016" layer="1"/>
 <contactref element="X8" pad="2"/>
-<wire x1="5.08" y1="53.3908" x2="12.7" y2="54.61" width="0" layer="19" extent="1-1"/>
+<wire x1="5.08" y1="53.3908" x2="11.4808" y2="53.3908" width="1.016" layer="1"/>
+<wire x1="11.4808" y1="53.3908" x2="12.7" y2="54.61" width="1.016" layer="1"/>
 </signal>
 <signal name="N$26">
@@
 <wire x1="15.24" y1="59.69" x2="12.7" y2="57.15" width="1.016" layer="1"/>
 <contactref element="X8" pad="1"/>
-<wire x1="5.08" y1="58.3946" x2="12.7" y2="57.15" width="0" layer="19" extent="1-1"/>
+<wire x1="5.08" y1="58.3946" x2="11.4554" y2="58.3946" width="1.016" layer="1"/>
+<wire x1="11.4554" y1="58.3946" x2="12.7" y2="57.15" width="1.016" layer="1"/>
 </signal>
 <signal name="N$28">
@@
 <wire x1="15.24" y1="40.64" x2="12.7" y2="43.18" width="1.016" layer="1"/>
 <contactref element="X9" pad="2"/>
-<wire x1="5.08" y1="41.9608" x2="12.7" y2="43.18" width="0" layer="19" extent="1-1"/>
+<wire x1="5.08" y1="41.9608" x2="11.4808" y2="41.9608" width="1.016" layer="1"/>
+<wire x1="11.4808" y1="41.9608" x2="12.7" y2="43.18" width="1.016" layer="1"/>
 </signal>
 <signal name="N$34">
@@
 <wire x1="15.24" y1="48.26" x2="12.7" y2="45.72" width="1.016" layer="1"/>
 <contactref element="X9" pad="1"/>
-<wire x1="5.08" y1="46.9646" x2="12.7" y2="45.72" width="0" layer="19" extent="1-1"/>
+<wire x1="5.08" y1="46.9646" x2="11.4554" y2="46.9646" width="1.016" layer="1"/>
+<wire x1="11.4554" y1="46.9646" x2="12.7" y2="45.72" width="1.016" layer="1"/>
 </signal>
 <signal name="N$36">
@@
 <wire x1="43.5178" y1="35.4" x2="49.53" y2="35.4" width="1.016" layer="1"/>
 <wire x1="49.53" y1="35.4" x2="50.8" y2="36.67" width="1.016" layer="1"/>
-<wire x1="50.8" y1="36.67" x2="54.61" y2="36.67" width="1.016" layer="1"/>
+<wire x1="50.8" y1="36.67" x2="53.34" y2="36.67" width="1.016" layer="1"/>
 </signal>
 <signal name="N$1">
