File: MCP23017 Boards/O8/EAGLE/MCP23017_O8_v1_01.brd (EAGLE design)
At the start: 90 x 90 mm, 79 parts, among them IC5 MCP23017SP, X4 057-016-0

Commit message: Update MCP23017_O8_v1_01.brd
Routing:
- net N$84: track 0.00 -> 79.7 mm
- net N$82: track 0.00 -> 69.2 mm
- net N$55: track 8.15 -> 50.1 mm
- net N$2: track 8.15 -> 48.4 mm
- net N$52: track 8.15 -> 46.6 mm
- net N$22: track 8.15 -> 43.4 mm
- net N$12: track 8.15 -> 40.5 mm
- net N$50: track 8.15 -> 37.4 mm
- net GND2: track 70.7 -> 98.9 mm
- net N$24: track 8.15 -> 34.7 mm
- net N$20: track 8.15 -> 33.9 mm
- net N$18: track 8.15 -> 33.9 mm
- net N$14: track 8.15 -> 30.0 mm
- net N$59: track 8.15 -> 29.9 mm
- net N$16: track 8.15 -> 29.5 mm
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